File: Vaimanika_H7/Vaimanika_H7.kicad_pcb (KiCad board)
At the start: 4 copper layers, 40 x 40 mm, 50 parts, among them J1 USB_C_Receptacle_USB2.0_16P, J2 Conn_01x08, J3 Conn_01x08, J4 +VLIPO, J5 GND, J6 Conn_01x08, J7 Conn_01x03, Q1 AO3400A, Q2 AO3401A, U2 TPS54302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

Commit message: 15-04-2026
Parts:
- removed C13: 75pF, Capacitor_SMD:C_0402_1005Metric
- removed D1: 1N4148, Diode_SMD:D_SOD-523
- added C12: 4.7uF, Capacitor_SMD:C_0603_1608Metric, B.Cu at (130.8, 88.7)
- added C17: 47uF, Capacitor_SMD:C_0805_2012Metric, B.Cu at (122.8, 75.5)
- added C18: 4.7uF, Capacitor_SMD:C_0603_1608Metric, B.Cu at (122.3, 79.9)
- added C19: 1uF, Capacitor_SMD:C_0402_1005Metric, B.Cu at (132.5, 77.8)
- added C20: 100nF, Capacitor_SMD:C_0402_1005Metric, B.Cu at (132.5, 80.2)
- added FPC2: AFC24-S40FIA-HF, New_Library:FPC-SMD_40P-P0.50_AFC24-S40FIA-HF, F.Cu at (140.7, 78.2)
- C14: value 10uF -> 75pF; footprint Capacitor_SMD:C_0805_2012Metric -> Capacitor_SMD:C_0402_1005Metric
- C15: value 47uF -> 1uF; footprint Capacitor_SMD:C_0805_2012Metric -> Capacitor_SMD:C_0402_1005Metric
- C16: value 10uF -> 100nF; footprint Capacitor_SMD:C_0805_2012Metric -> Capacitor_SMD:C_0402_1005Metric
- C3, R1, R2, R4: moved to B.Cu
- moved R5 135.7 mm to (194.1, 80.9), turned to -90 degrees
- moved R3 133.5 mm to (191.6, 78.1)
- moved Q1 127.5 mm to (195.0, 77.2), turned to 90 degrees
- moved R1 93.9 mm to (149.1, 79.3), turned to 90 degrees
- moved R4 93.5 mm to (150.9, 78.0)
- moved R2 92.4 mm to (149.1, 76.5), turned to 90 degrees
- moved C3 84.9 mm to (151.1, 80.0), turned to -90 degrees
- moved H6 18.5 mm to (124.7, 71.5)
- moved C16 13.6 mm to (127.4, 89.2), turned to -90 degrees
- moved C14 8.61 mm to (139.4, 90.5), turned to 0 degrees
- moved C15 7.73 mm to (128.9, 89.2), turned to -90 degrees
- moved R20 6.53 mm to (126.7, 75.5), turned to 0 degrees
- moved H5 1.20 mm to (149.3, 96.0)
Connections:
- C14 pad 1: +5VBAT -> Net-(C14-Pad1)
- C14 pad 2: GND -> Net-(U2-FB)
- C15 pad 2: Net-(C15-Pad2) -> GND
- C16 pad 1: +5VFIL -> +5VBAT
- R17 pad 1: Net-(C13-Pad1) -> Net-(C14-Pad1)
- R18 pad 2: Net-(C13-Pad1) -> Net-(C14-Pad1)
- R20 pad 1: +5VFIL -> Net-(C17-Pad1)
- R20 pad 2: Net-(C15-Pad2) -> +5VFIL
Routing:
- net +5VFIL: track 17.4 -> 26.1 mm
- net GND: track 25.4 -> 29.4 mm
- net Net-(R1-Pad2): track 0.00 -> 3.12 mm
- net +5VBAT: track 28.7 -> 31.8 mm
- net +VIN: track 21.1 -> 24.1 mm
- net Net-(C14-Pad1): track 0.00 -> 2.95 mm
- net Net-(C13-Pad1): track 2.94 -> 0.00 mm
- net Net-(C17-Pad1): track 0.00 -> 2.12 mm
- net Net-(C15-Pad2): track 1.95 -> 0.00 mm
- net ADC_VOLTAGE: track 0.00 -> 1.70 mm

Commit message: 23-04-2026
Routing:
- net GND: vias 1 -> 30
Changed lines of the file:
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@@
+	)
+	(via
+		(at 120.83 99.861627)
+		(size 0.6)
+		(drill 0.3)
+		(layers "F.Cu" "B.Cu")
+		(free yes)
+		(net 1)
+	)
+	(via
+		(at 120.87 65.58)
+		(size 0.6)
+		(drill 0.3)
+		(layers "F.Cu" "B.Cu")
+		(free yes)
+		(net 1)
+	)
+	(via
+		(at 159.07 93.511627)
+		(size 0.6)
+		(drill 0.3)
+		(layers "F.Cu" "B.Cu")
+		(free yes)
+		(net 1)
+	)
+	(via
+		(at 151.078373 99.81)
+		(size 0.6)
+		(drill 0.3)
+		(layers "F.Cu" "B.Cu")
+		(free yes)
+		(net 1)
+	)
+	(via
+		(at 159.06 97.511627)
+		(size 0.6)
+		(drill 0.3)
+		(layers "F.Cu" "B.Cu")
+		(free yes)
+		(net 1)
+	)
+	(via
+		(at 120.85 81.561627)
+		(size 0.6)
+		(drill 0.3)
+		(layers "F.Cu" "B.Cu")
+		(free yes)
+		(net 1)
+	)
+	(via
+		(at 120.85 93.531627)
+		(size 0.6)
+		(drill 0.3)
+		(layers "F.Cu" "B.Cu")
+		(free yes)
+		(net 1)
+	)
+	(via
+		(at 159.05 99.841627)
+		(size 0.6)
+		(drill 0.3)
+		(layers "F.Cu" "B.Cu")
+		(free yes)
+		(net 1)
+	)
+	(via
+		(at 159.078373 61.6)
+		(size 0.6)
+		(drill 0.3)
+		(layers "F.Cu" "B.Cu")
+		(free yes)
+		(net 1)
+	)
+	(via
+		(at 159.06 85.531627)
+		(size 0.6)
+		(drill 0.3)
+		(layers "F.Cu" "B.Cu")
+		(free yes)
+		(net 1)
+	)
+	(via
+		(at 120.84 85.551627)
+		(size 0.6)
+		(drill 0.3)
+		(layers "F.Cu" "B.Cu")
+		(free yes)
+		(net 1)
+	)
+	(via
+		(at 120.86 77.571627)
+		(size 0.6)
+		(drill 0.3)
+		(layers "F.Cu" "B.Cu")
+		(free yes)
+		(net 1)
+	)
+	(via
+		(at 120.87 61.62)
+		(size 0.6)
+		(drill 0.3)
+		(layers "F.Cu" "B.Cu")
+		(free yes)
+		(net 1)
+	)
+	(via
+		(at 120.84 89.531627)
+		(size 0.6)
+		(drill 0.3)
+		(layers "F.Cu" "B.Cu")
+		(free yes)
+		(net 1)
+	)
+	(via
+		(at 159.09 65.56)
+		(size 0.6)
+		(drill 0.3)
+		(layers "F.Cu" "B.Cu")
+		(free yes)
+		(net 1)
+	)
+	(via
+		(at 120.86 73.571627)
+		(size 0.6)
+		(drill 0.3)
+		(layers "F.Cu" "B.Cu")
+		(free yes)
+		(net 1)
 	)
 	(via
@@
 		(net 1)
 	)
+	(via
+		(at 131.118373 99.79)
+		(size 0.6)
+		(drill 0.3)
+		(layers "F.Cu" "B.Cu")
+		(free yes)
+		(net 1)
+	)
+	(via
+		(at 120.84 97.531627)
+		(size 0.6)
+		(drill 0.3)
+		(layers "F.Cu" "B.Cu")
+		(free yes)
+		(net 1)
+	)
+	(via
+		(at 159.07 81.541627)
+		(size 0.6)
+		(drill 0.3)
+		(layers "F.Cu" "B.Cu")
+		(free yes)
+		(net 1)
+	)
+	(via
+		(at 159.08 69.551627)
+		(size 0.6)
+		(drill 0.3)
+		(layers "F.Cu" "B.Cu")
+		(free yes)
+		(net 1)
+	)
+	(via
+		(at 155.09 61.67)
+		(size 0.6)
+		(drill 0.3)
+		(layers "F.Cu" "B.Cu")
+		(free yes)
+		(net 1)
+	)
+	(via
+		(at 123.138373 61.64)
+		(size 0.6)
+		(drill 0.3)
+		(layers "F.Cu" "B.Cu")
+		(free yes)
+		(net 1)
+	)
+	(via
+		(at 147.078373 99.81)
+		(size 0.6)
+		(drill 0.3)
+		(layers "F.Cu" "B.Cu")
+		(free yes)
+		(net 1)
+	)
+	(via
+		(at 155.07 99.82)
+		(size 0.6)
+		(drill 0.3)
+		(layers "F.Cu" "B.Cu")
+		(free yes)
+		(net 1)
+	)
+	(via
+		(at 127.138373 61.65)
+		(size 0.6)
+		(drill 0.3)
+		(layers "F.Cu" "B.Cu")
+		(free yes)
+		(net 1)
+	)
+	(via
+		(at 127.118373 99.8)
+		(size 0.6)
+		(drill 0.3)
+		(layers "F.Cu" "B.Cu")
+		(free yes)
+		(net 1)
+	)
+	(via
+		(at 159.06 89.511627)
+		(size 0.6)
+		(drill 0.3)
+		(layers "F.Cu" "B.Cu")
+		(free yes)
+		(net 1)
+	)
+	(via
+		(at 123.118373 99.79)
+		(size 0.6)
+		(drill 0.3)
+		(layers "F.Cu" "B.Cu")
+		(free yes)
+		(net 1)
+	)
+	(via
+		(at 120.86 69.571627)
+		(size 0.6)
+		(drill 0.3)
+		(layers "F.Cu" "B.Cu")
+		(free yes)
+		(net 1)
+	)
