File: Vaimanika_H7/Vaimanika_H7.kicad_pcb (KiCad board)
At the start: 4 copper layers, 40 x 40 mm, 61 parts, among them CN1 WAFER-GH1.25-3PWB, J1 USB_C_Receptacle_USB2.0_16P, J2 Conn_01x08, J3 Conn_01x08, J4 +VLIPO, J5 GND, J6 Conn_01x08, J7 Conn_01x03, Q1 AO3400A, Q2 AO3401A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

Commit message: 02-05-2026
Parts:
- U7, U8, U9: value WAFER-GH1.25-4PWB -> WAFER-GH1.25-4PLB; footprint New_Library:CONN-SMD_4P-P1.25_XUNPU_WAFER-GH1.25-4PWB -> New_Library:CONN-SMD_4P-P1.25_XUNPU_WAFER-GH1.25-4PLB
- moved U9 38.6 mm to (131.8, 84.5)
- moved U8 34.2 mm to (147.7, 84.3), turned to 0 degrees
- moved U7 26.6 mm to (132.2, 94.2), turned to -90 degrees
- moved CN1 26.3 mm to (156.1, 84.3), turned to 90 degrees
- moved U6 2.31 mm to (156.0, 75.0)
- moved U3 1.22 mm to (140.9, 86.9)
- moved J1 1.22 mm to (141.2, 96.9)
- moved R12 1.22 mm to (139.7, 90.7)
- moved R13 1.22 mm to (142.7, 90.7)
- moved U5 0.56 mm to (123.9, 88.0)
Routing:
- net +5VBUS: track 28.5 -> 49.1 mm, vias 4 -> 5
- net GND: track 44.0 -> 41.2 mm
- net Net-(R11-Pad1): track 2.27 -> 2.77 mm

Commit message: 02-05-2026
Parts:
- added J8: Conn_01x02, Connector_PinHeader_1.27mm:PinHeader_1x02_P1.27mm_Vertical, F.Cu at (158.2, 82.9)
- moved Q1 40.6 mm to (154.7, 81.8)
- moved R5 40.0 mm to (154.3, 84.5), turned to 0 degrees
- moved R3 39.5 mm to (152.3, 82.2), turned to -90 degrees
- moved U7 18.6 mm to (148.6, 85.6), turned to 0 degrees
- moved U8 18.4 mm to (132.2, 94.2), turned to -90 degrees
- moved CN1 4.71 mm to (156.1, 89.1)
- moved J4 1.88 mm to (157.1, 74.7)
- moved J5 1.88 mm to (157.1, 71.2)
Routing:
- net PIN_B+: track 62.7 -> 199.3 mm, vias 4 -> 15
- net CAN_H: track 0.00 -> 56.1 mm, vias 0 -> 3
- net CAN_L: track 0.00 -> 52.9 mm, vias 0 -> 3
- net I2C2_SDA: track 0.00 -> 36.3 mm, vias 0 -> 2
- net I2C2_SCL: track 0.00 -> 35.0 mm, vias 0 -> 2
- net UART2_TX: track 0.00 -> 33.8 mm, vias 0 -> 2
- net UART2_RX: track 0.00 -> 32.3 mm, vias 0 -> 2
- net USART1_TX: track 0.00 -> 27.0 mm, vias 0 -> 2
- net SCL_BARO: track 0.00 -> 23.3 mm, vias 0 -> 2
- net USART1_RX: track 0.00 -> 22.0 mm, vias 0 -> 2
- net SDA_BARO: track 0.00 -> 21.6 mm, vias 0 -> 2
- net ADC: track 0.00 -> 18.4 mm, vias 0 -> 2
- net USART6_RX: track 0.00 -> 7.92 mm
- net Net-(U2-FB): track 3.57 -> 11.0 mm, vias 1 -> 2
- net USART6_TX: track 0.00 -> 7.34 mm
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Other:
- board text added: "5V"
- board text added: "ADC"
- board text added: "CAN"
- board text added: "G"
- board text added: "I2C1"
- board text added: "I2C2"
- board text added: "M1"
- board text added: "M2"
- board text added: "M3"
- board text added: "M4"
- board text added: "M5"
- board text added: "M6"
- board text added: "M7"
- board text added: "M8"
- board text added: "S"
- board text added: "UART"

Commit message: 02-05-2026
Parts:
- removed J7: Conn_01x03, Connector_PinHeader_2.54mm:PinHeader_1x03_P2.54mm_Vertical
- J1: value USB_C_Receptacle_USB2.0_16P -> TYPE-C 16PIN 2MD; footprint Connector_USB:USB_C_Receptacle_GCT_USB4105-xx-A_16P_TopMnt_Horizontal -> New_Library:USB-C-SMD_TYPE-C-16PIN-2MD-073
- J2, J3, J6: value Conn_01x08 -> Conn_01x09; footprint Connector_PinHeader_2.54mm:PinHeader_1x08_P2.54mm_Vertical -> Connector_PinHeader_2.54mm:PinHeader_1x09_P2.54mm_Vertical
- moved J1 1.31 mm to (141.2, 95.6)
- turned R12 to -90 degrees
- turned R13 to -90 degrees
Connections:
- R12 pad 1: Net-(J1-CC1) -> GND
- R12 pad 2: GND -> Net-(J1-CC1)
- R13 pad 1: Net-(J1-CC2) -> GND
- R13 pad 2: GND -> Net-(J1-CC2)
Routing:
- net PIN_B+: track 199.3 -> 203.2 mm

Commit message: 05-05-2026
Parts:
- added G***: LOGO, LOGO, B.Cu at (142.6, 96.1)
Other:
- board text added: "P.B. Rev 1.0"
- board text added: "RX"
- board text added: "Vaimanika Aerospace"

Commit message: 18-05-2026
Routing:
- net GND: vias 35 -> 57
Other:
- board text added: "B+"
- board text added: "B-"
- board text added: "UART1"
- board text added: "UART2"
- board text added: "UART6"
- board text removed: "UART"

Commit message: 21-05-2026
Parts:
- removed the G*** at (142.6, 96.1)
- added G***: LOGO, LOGO, F.Cu at (149.5, 91.5)
- added G***: LOGO, LOGO, B.Cu at (144.5, 97.6)
Routing:
- net CAN_L: track 52.9 -> 50.9 mm
- net GND: vias 57 -> 58
Other:
- board text added: "+"
- board text added: "-"
- board text added: "AEROSPACE"
- board text added: "VA-VEG_H7-FC-PWR-R1.0"
- board text added: "VAIMANIKA"
- board text removed: "P.B. Rev 1.0"
- board text removed: "Vaimanika Aerospace"

Commit message: 21-05-2026
Other:
- board text added: "P IN"
Changed lines of the file:
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@@
 			)
 		)
+		(property "LCSC" "C492401"
+			(at 0 0 180)
+			(unlocked yes)
+			(layer "F.Fab")
+			(hide yes)
+			(effects
+				(font
+					(size 1 1)
+					(thickness 0.15)
+				)
+			)
+		)
 		(property ki_fp_filters "Connector*:*_1x??_*")
 		(sheetname "/")
@@
 			)
 		)
+		(property "LCSC" "C492408"
+			(at 0 0 90)
+			(unlocked yes)
+			(layer "F.Fab")
+			(hide yes)
+			(effects
+				(font
+					(size 1 1)
+					(thickness 0.15)
+				)
+			)
+		)
 		(property ki_fp_filters "Connector*:*_1x??_*")
 		(sheetname "/")
@@
 			)
 		)
+		(property "LCSC" "C492408"
+			(at 0 0 270)
+			(unlocked yes)
+			(layer "B.Fab")
+			(hide yes)
+			(effects
+				(font
+					(size 1 1)
+					(thickness 0.15)
+				)
+				(justify mirror)
+			)
+		)
 		(property ki_fp_filters "Connector*:*_1x??_*")
 		(sheetname "/")
@@
 			)
 		)
+		(property "LCSC" "C492408"
+			(at 0 0 270)
+			(unlocked yes)
+			(layer "B.Fab")
+			(hide yes)
+			(effects
+				(font
+					(size 1 1)
+					(thickness 0.15)
+				)
+				(justify mirror)
+			)
+		)
 		(property ki_fp_filters "Connector*:*_1x??_*")
 		(sheetname "/")
@@
 		)
 	)
+	(gr_text "P IN"
+		(at 152.56 71.24 90)
+		(layer "B.SilkS")
+		(effects
+			(font
+				(size 1 1)
+				(thickness 0.125)
+			)
+			(justify left bottom mirror)
+		)
+	)
 	(gr_text "VAIMANIKA"
 		(at 141.508093 97.712195 0)
@@
 	)
 	(via
-		(at 152.37 68.7)
+		(at 153.14 68.72)
 		(size 0.6)
 		(drill 0.3)
@@
 		(polygon
 			(pts
-				(xy 127.42 64.14) (xy 152.13 64.14) (xy 152.13 69.6) (xy 151.95 69.78) (xy 127.42 69.78)
+				(xy 127.42 64.14) (xy 152.37 64.14) (xy 152.37 69.85) (xy 153.35 69.78) (xy 127.42 69.78)
 			)
 		)
