File: Vaimanika_H7/Vaimanika_H7.kicad_sch (KiCad schematic)
At the start: 44 parts, among them J1 USB_C_Receptacle_USB2.0_16P, Q1 AO3400A, Q2 AO3401A, U3 TPS54302, U4 TPS54302, U5 USBLC6-2P6

Commit message: 28-03-2025
Parts:
- removed TP8: TestPoint, TestPoint:TestPoint_Pad_D1.0mm, symbol Connector:TestPoint
- added C14, C16: 10uF, Capacitor_SMD:C_0805_2012Metric, symbol Device:C
- added C15: 47uF, Capacitor_SMD:C_0805_2012Metric, symbol Device:C
- added D1: 1N4148, Diode_SMD:D_SOD-523, symbol Diode:1N4148
- added H1, H2, H3, H4: MountingHole, MountingHole:MountingHole_4.3mm_M4, symbol Mechanical:MountingHole
- added H5: MountingHole, MountingHole:MountingHole_2.7mm_M2.5_DIN965, symbol Mechanical:MountingHole
- added H6: MountingHole, MountingHole:MountingHole_2.7mm_M2.5, symbol Mechanical:MountingHole
- added J2, J3, J6: Conn_01x08, Connector_PinHeader_2.54mm:PinHeader_1x08_P2.54mm_Vertical, symbol Connector_Generic:Conn_01x08
- added J4: +VLIPO, New_Library:SolderPads_1x1_2.5_3.5, symbol Connector:Conn_01x01_Socket
- added J5: GND, New_Library:SolderPads_1x1_2.5_3.5, symbol Connector:Conn_01x01_Socket
- added J7: Conn_01x03, Connector_PinHeader_2.54mm:PinHeader_1x03_P2.54mm_Vertical, symbol Connector_Generic:Conn_01x03
- added L3: 10uH, Inductor_SMD:L_Chilisin_BMRB00060612, symbol Device:L
- added R20: 1, Resistor_SMD:R_0805_2012Metric, symbol Device:R
- added R3: 100, Resistor_SMD:R_0402_1005Metric, symbol Device:R
- added R5: 10K, Resistor_SMD:R_0402_1005Metric, symbol Device:R
- D2: renamed from D3; value SS24FL -> SS34; footprint Diode_SMD:D_SOD-123F -> Diode_SMD:D_SMA; LCSC C894433 -> C8678
- D3: renamed from D5; value SS24FL -> SS34; footprint Diode_SMD:D_SOD-123F -> Diode_SMD:D_SMA; LCSC C894433 -> C8678
- Q1: BOARD SENSOR -> POWER
- renumbered C3 to C1, C17 to C10, C18 to C11, C22 to C12, C23 to C13, C4 to C2, C44 to C3, C8 to C4, C9 to C5, C13 to C6, C14 to C7, C15 to C8, C16 to C9, R25 to R1, R5 to R10, R6 to R11, R7 to R12, R8 to R13, R10 to R14, R11 to R15, R12 to R16, R13 to R17, R14 to R18, R15 to R19, R26 to R2, R32 to R21, R28 to R4, R1 to R6, R2 to R7, R3 to R8, R4 to R9, U3 to U1, U4 to U2, U5 to U3
Connections:
- net +5V: now also D1.1 (K), J2.1 (Pin_1), J2.2 (Pin_2), J2.3 (Pin_3), J2.4 (Pin_4), J2.5 (Pin_5), J2.6 (Pin_6), J2.7 (Pin_7), J2.8 (Pin_8), J7.2 (Pin_2)
- net +5VBAT: now also C14.1, C15.1, L3.1; no longer D2.2 (A)
- net +VLIPO: now also J4.1 (Pin_1)
- net BUZZER: now also R3.1; no longer Q1.1 (G)
- net GND: now also C14.2, C16.2, J3.1 (Pin_1), J3.2 (Pin_2), J3.3 (Pin_3), J3.4 (Pin_4), J3.5 (Pin_5), J3.6 (Pin_6), J3.7 (Pin_7), J3.8 (Pin_8), J5.1 (Pin_1), J7.1 (Pin_1), R5.2
- net PIN_B-: now also D1.2 (A)
- new net: C15.2, R20.2
- new net: Q1.1 (G), R3.2, R5.1
- new net +5VFIL: C16.1, D2.2 (A), L3.2, R20.1
Other:
- note added: "Ports and I/Os"
- note added: "π Filter"
- moved on the sheet: Q1

Commit message: 10-04-2026
Other:
- moved on the sheet: C14, C15, C16, L3, R20

Commit message: 15-04-2026
Parts:
- removed C14: 10uF, Capacitor_SMD:C_0805_2012Metric, symbol Device:C
- removed D1: 1N4148, Diode_SMD:D_SOD-523, symbol Diode:1N4148
- added C12, C18: 4.7uF, Capacitor_SMD:C_0603_1608Metric, symbol Device:C
- added C15, C19: 1uF, Capacitor_SMD:C_0402_1005Metric, symbol Device:C
- added C20: 100nF, Capacitor_SMD:C_0402_1005Metric, symbol Device:C
- added FPC2: AFC24-S40FIA-HF, New_Library:FPC-SMD_40P-P0.50_AFC24-S40FIA-HF, symbol New_Library:AFC24-S40FIA-HF
- C16: value 10uF -> 100nF; footprint Capacitor_SMD:C_0805_2012Metric -> Capacitor_SMD:C_0402_1005Metric; LCSC C95841 -> C60474
- renumbered C12 to C13, C13 to C14, C15 to C17
Connections:
- net +5VBAT: now also C16.1, C12.1, C15.1; no longer C17.1
- net +5VFIL: now also R20.2, C18.1, C19.1, C20.1; no longer C16.1, R20.1
- net GND: now also C17.2, C12.2, C15.2, C18.2, C19.2, C20.2
- new net: C17.1, R20.1
Other:
- moved on the sheet: C17, D4, F1, J2, J3, J4, J5, L3, Q2, R20, R21

Commit message: 23-04-2026
Connections:
- net +5V: now also FPC2.35, FPC2.36, FPC2.37, FPC2.38
- net BUZZER: now also FPC2.9
- net GND: now also FPC2.12, FPC2.25, FPC2.28, FPC2.31, FPC2.32, FPC2.33, FPC2.34, FPC2.39, FPC2.40, FPC2.41, FPC2.42
- net USB_D+: now also FPC2.30
- net USB_D-: now also FPC2.29
- net MOTOR8: now reaches FPC2.1
- net RX_PPM: now reaches FPC2.10
- net ADC: now reaches FPC2.11
- net USART6_RX: now reaches FPC2.13
- net USART6_TX: now reaches FPC2.14
- net UART2_RX: now reaches FPC2.15
- net UART2_TX: now reaches FPC2.16
- net USART1_RX: now reaches FPC2.19
- net MOTOR7: now reaches FPC2.2
- net USART1_TX: now reaches FPC2.20
- net I2C2_SDA: now reaches FPC2.21
- net I2C2_SCL: now reaches FPC2.22
- net SCL_BARO: now reaches FPC2.23
- net SDA_BARO: now reaches FPC2.24
- net CAN_L: now reaches FPC2.26
- net CAN_H: now reaches FPC2.27
- net MOTOR6: now reaches FPC2.3
- net MOTOR5: now reaches FPC2.4
- net MOTOR4: now reaches FPC2.5
- net MOTOR3: now reaches FPC2.6
- net MOTOR2: now reaches FPC2.7
- net MOTOR1: now reaches FPC2.8
Other:
- note added: "Pin 7 and 8 are Empty could be sued for different purpose adn for now conencted to Gnd"

Commit message: 01-05-2026
Parts:
- added CN1: WAFER-GH1.25-3PWB, New_Library:CONN-TH_3P-P1.25_GH1.25, symbol New_Library:WAFER-GH1.25-3PWB
- added U4, U5, U6, U7, U8, U9: WAFER-GH1.25-4PWB, New_Library:CONN-SMD_4P-P1.25_XUNPU_WAFER-GH1.25-4PWB, symbol New_Library:WAFER-GH1.25-4PWB
- renumbered D2 to D1, D3 to D2, D4 to D3, FPC2 to FPC1
Connections:
- net +5V: now also CN1.1, U4.1, U5.1, U6.1, U7.1, U8.1, U9.1
- net ADC: now also CN1.2
- net CAN_H: now also U6.2
- net CAN_L: now also U6.3
- net GND: now also CN1.3, CN1.4, CN1.5, U4.4, U4.5, U4.6, U5.4, U5.5, U5.6, U6.4, U6.5, U6.6, U7.4, U7.5, U7.6, U8.4, U8.5, U8.6, U9.4, U9.5, U9.6
- net I2C2_SCL: now also U5.2
- net I2C2_SDA: now also U5.3
- net MOTOR1: now also J6.1 (Pin_1)
- net MOTOR2: now also J6.2 (Pin_2)
- net MOTOR3: now also J6.3 (Pin_3)
- net MOTOR4: now also J6.4 (Pin_4)
- net MOTOR5: now also J6.5 (Pin_5)
- net MOTOR6: now also J6.6 (Pin_6)
- net MOTOR7: now also J6.7 (Pin_7)
- net MOTOR8: now also J6.8 (Pin_8)
- net RX_PPM: now also J7.3 (Pin_3)
- net SCL_BARO: now also U4.2
- net SDA_BARO: now also U4.3
- net UART2_RX: now also U8.3
- net UART2_TX: now also U8.2
- net USART1_RX: now also U9.3
- net USART1_TX: now also U9.2
- net USART6_RX: now also U7.3
- net USART6_TX: now also U7.2
- no-connect marks 2 -> 4

Commit message: 02-05-2026
Parts:
- removed U7, U8, U9: WAFER-GH1.25-4PWB, New_Library:CONN-SMD_4P-P1.25_XUNPU_WAFER-GH1.25-4PWB, symbol New_Library:WAFER-GH1.25-4PWB
- added U7, U8, U9: WAFER-GH1.25-4PLB, New_Library:CONN-SMD_4P-P1.25_XUNPU_WAFER-GH1.25-4PLB, symbol New_Library:WAFER-GH1.25-4PLB
Connections:
- net +5V: now also U7.1, U8.1, U9.1
- net GND: now also U7.4, U7.5, U7.6, U8.4, U8.5, U8.6, U9.4, U9.5, U9.6
- net UART2_RX: now also U8.3
- net UART2_TX: now also U8.2
- net USART1_RX: now also U9.3
- net USART1_TX: now also U9.2
- net USART6_RX: now also U7.3
- net USART6_TX: now also U7.2

Commit message: 02-05-2026
Parts:
- added J8: Conn_01x02, Connector_PinHeader_1.27mm:PinHeader_1x02_P1.27mm_Vertical, symbol Connector_Generic:Conn_01x02
Connections:
- net +5V: now also J8.1 (Pin_1)
- net PIN_B-: now also J8.2 (Pin_2)
Changed lines of the file:
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@@
 		)
 	)
+	(global_label "PIN_B-"
+		(shape input)
+		(at 248.92 35.56 180)
+		(fields_autoplaced yes)
+		(effects
+			(font
+				(size 1.27 1.27)
+			)
+			(justify right)
+		)
+		(property "Intersheetrefs" "${INTERSHEET_REFS}"
+			(at 238.9195 35.56 0)
+			(effects
+				(font
+					(size 1.27 1.27)
+				)
+				(justify right)
+				(hide yes)
+			)
+		)
+	)
 	(global_label "CAN_H"
 		(shape input)
@@
 		)
 	)
+	(global_label "PIN_B+"
+		(shape input)
+		(at 248.92 33.02 180)
+		(fields_autoplaced yes)
+		(effects
+			(font
+				(size 1.27 1.27)
+			)
+			(justify right)
+		)
+		(property "Intersheetrefs" "${INTERSHEET_REFS}"
+			(at 238.9195 33.02 0)
+			(effects
+				(font
+					(size 1.27 1.27)
+				)
+				(justify right)
+				(hide yes)
+			)
+		)
+	)
 	(global_label "ADC"
 		(shape input)
@@
 					(unit 1)
 				)
+			)
+		)
+	)
+	(symbol
+		(lib_id "Connector_Generic:Conn_01x02")
+		(at 254 33.02 0)
+		(unit 1)
+		(exclude_from_sim no)
+		(in_bom yes)
+		(on_board yes)
+		(dnp no)
+		(property "Reference" "J8"
+			(at 255.27 33.782 0)
+			(effects
+				(font
+					(size 1.27 1.27)
+				)
+				(justify left)
+			)
+		)
+		(property "Value" "Conn_01x02"
+			(at 245.364 39.116 0)
+			(effects
+				(font
+					(size 1.27 1.27)
+				)
+				(justify left)
+			)
+		)
+		(property "Footprint" "Connector_PinHeader_1.27mm:PinHeader_1x02_P1.27mm_Vertical"
+			(at 254 33.02 0)
+			(effects
+				(font
+					(size 1.27 1.27)
+				)
+				(hide yes)
+			)
+		)
+		(property "Datasheet" "~"
+			(at 254 33.02 0)
+			(effects
+				(font
+					(size 1.27 1.27)
+				)
+				(hide yes)
+			)
+		)
+		(property "Description" "Generic connector, single row, 01x02, script generated (kicad-library-utils/schlib/autogen/connector/)"
+			(at 254 33.02 0)
+			(effects
+				(font
+					(size 1.27 1.27)
+				)
+				(hide yes)
+			)
+		)
+		(pin "2"
+		)
+		(pin "1"
+		)
+		(instances
+			(project ""
+				(path "/0142fa91-cde5-4e00-8a71-4202316295cd"
+					(reference "J8")
+					(unit 1)
+				)

Commit message: 02-05-2026
Parts:
- removed J1: USB_C_Receptacle_USB2.0_16P, Connector_USB:USB_C_Receptacle_GCT_USB4105-xx-A_16P_TopMnt_Horizontal, symbol Connector:USB_C_Receptacle_USB2.0_16P
- removed J2, J3, J6: Conn_01x08, Connector_PinHeader_2.54mm:PinHeader_1x08_P2.54mm_Vertical, symbol Connector_Generic:Conn_01x08
- removed J7: Conn_01x03, Connector_PinHeader_2.54mm:PinHeader_1x03_P2.54mm_Vertical, symbol Connector_Generic:Conn_01x03
- added J1: TYPE-C 16PIN 2MD, New_Library:USB-C-SMD_TYPE-C-16PIN-2MD-073, symbol New_Library:TYPE-C16PIN2MD
- added J2, J3, J6: Conn_01x09, Connector_PinHeader_2.54mm:PinHeader_1x09_P2.54mm_Vertical, symbol Connector_Generic:Conn_01x09
Connections:
- net +5V: now also J2.1 (Pin_1), J2.2 (Pin_2), J2.3 (Pin_3), J2.4 (Pin_4), J2.5 (Pin_5), J2.6 (Pin_6), J2.7 (Pin_7), J2.8 (Pin_8), J2.9 (Pin_9)
- net +5VBUS: now also J1.A4B9 (VBUS), J1.B4A9 (VBUS)
- net GND: now also R12.1, R13.1, J1.13 (EH), J1.14 (EH), J1.A1B12 (GND), J1.B1A12 (GND), J3.1 (Pin_1), J3.2 (Pin_2), J3.3 (Pin_3), J3.4 (Pin_4), J3.5 (Pin_5), J3.6 (Pin_6), J3.7 (Pin_7), J3.8 (Pin_8), J3.9 (Pin_9); no longer R12.2, R13.2
- net MOTOR1: now also J6.1 (Pin_1)
- net MOTOR2: now also J6.2 (Pin_2)
- net MOTOR3: now also J6.3 (Pin_3)
- net MOTOR4: now also J6.4 (Pin_4)
- net MOTOR5: now also J6.5 (Pin_5)
- net MOTOR6: now also J6.6 (Pin_6)
- net MOTOR7: now also J6.7 (Pin_7)
- net MOTOR8: now also J6.8 (Pin_8)
- net RX_PPM: now also J6.9 (Pin_9)
- net USB_CON_D+: now also J1.A6 (Dp1), J1.B6 (Dp2)
- net USB_CON_D-: now also J1.A7 (Dn1), J1.B7 (Dn2)
- new net: J1.A5 (CC1), R12.2
- new net: J1.B5 (CC2), R13.2
Other:
- moved on the sheet: R12, R13
