File: Vaimanika_H7_Sensor/Vaimanika_H7_Sensor.kicad_pcb (KiCad board)
At the start: 8 copper layers, 45 x 45 mm, 68 parts, among them SW1 TS-1088-AR02016, U1 TCAN334G, U2 STM32H743VITx, U3 NCP163ASN330T1G, U4 MS5611-01BA, U5 ICM-42688-P, U6 ICM-42688-P, U7 W25Q128JVS, U8 RT9080-33GJ5, U9 BMI088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

Commit message: 12-03-2026-02nd
Connections:
- U2 pad 15: unconnected-(U2-PC0-Pad15) -> IMU2_INT1
- U2 pad 35: IMU2_INT1 -> unconnected-(U2-PB1-Pad35)
Routing:
- net IMU2_INT3: track 0.00 -> 6.28 mm, vias 0 -> 2
- net IMU2_CSB2: track 0.00 -> 5.06 mm, vias 0 -> 2
- net IMU2_INT1: track 0.00 -> 4.23 mm, vias 0 -> 2

Commit message: 12-03-2026-03rd
Parts:
- TP1, TP2: moved to F.Cu
- moved C14 109.6 mm to (44.5, 41.5)
- moved U7 76.3 mm to (113.4, 69.4)
- moved C21 40.6 mm to (123.1, 80.6), turned to -90 degrees
- moved FB3 39.4 mm to (121.8, 80.6), turned to 90 degrees
- moved C18 37.5 mm to (120.5, 80.6), turned to -90 degrees
- moved FB2 33.6 mm to (119.6, 77.0), turned to 0 degrees
- moved C9 32.9 mm to (119.9, 78.6)
- moved FB7 30.4 mm to (122.7, 70.7), turned to 90 degrees
- moved C29 30.2 mm to (123.9, 70.7), turned to -90 degrees
- moved C19 22.9 mm to (134.4, 74.1), turned to 90 degrees
- moved FB5 22.1 mm to (133.2, 74.2), turned to -90 degrees
- moved U4 22.0 mm to (115.1, 79.4)
- moved C22 20.9 mm to (132.0, 74.1), turned to 90 degrees
- moved C10 17.0 mm to (135.0, 79.5)
- moved FB4 16.5 mm to (135.5, 77.9), turned to 180 degrees
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Routing:
- net SPI4_SCLK: track 0.00 -> 10.5 mm, vias 0 -> 3
- net CS_FLASH: track 0.00 -> 9.65 mm, vias 0 -> 1
- net SPI4_MISO: track 13.3 -> 21.1 mm, vias 3 -> 4
- net SPI4_MOSI: track 3.54 -> 7.68 mm, vias 2 -> 3
- net IMU2_INT2: track 0.00 -> 2.47 mm
Other:
- board text removed: "IMU 1"

Commit message: 28-03-2025
Parts:
- removed TF1: TF-CARD H1.8, New_Library:TF-SMD_TF-CARD-H1.8
- added SD1: TF-027-H300, New_Library:TF-SMD_HYCW104-TF08-375B, B.Cu at (111.8, 89.7)
- added TP3: TestPoint, TestPoint:TestPoint_Pad_D1.0mm, B.Cu at (110.8, 80.6)
- R9, U1, Y1: moved to B.Cu
- moved C11 107.2 mm to (124.9, 84.6), turned to 180 degrees
- moved C13 103.7 mm to (125.3, 81.7), turned to 90 degrees
- moved R9 97.4 mm to (117.9, 89.5)
- moved U8 95.8 mm to (134.5, 84.0), turned to 90 degrees
- moved U3 93.0 mm to (128.2, 84.0), turned to 90 degrees
- moved R2 89.2 mm to (115.5, 78.5), turned to 90 degrees
- moved R3 88.0 mm to (112.9, 81.5), turned to 180 degrees
- moved Y1 85.8 mm to (123.2, 63.1), turned to -135 degrees
- moved SW1 82.1 mm to (130.2, 67.7)
- moved C14 81.1 mm to (115.8, 80.0), turned to 0 degrees
- moved U1 76.5 mm to (109.8, 70.3), turned to 180 degrees
- moved G*** 3.62 mm to (140.3, 95.2)
- moved U4 2.87 mm to (112.6, 78.0), turned to 180 degrees
- moved C18 0.62 mm to (121.1, 80.6)
- moved C21 0.62 mm to (123.7, 80.6)
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Connections:
- U2 pad 7: SD_CD -> unconnected-(U2-PC13-Pad7)
Routing:
- net SD_CMD: track 0.00 -> 14.0 mm, vias 0 -> 2
- net SD_DAT0: track 0.00 -> 13.7 mm, vias 0 -> 2
- net SD_DAT1: track 0.00 -> 13.6 mm, vias 0 -> 2
- net SDA_BARO: track 0.00 -> 12.7 mm, vias 0 -> 2
- net SCL_BARO: track 0.00 -> 11.8 mm, vias 0 -> 2
- net SD_CLK: track 0.00 -> 11.1 mm, vias 0 -> 2
- net SD_DAT3: track 0.00 -> 10.2 mm, vias 0 -> 2
- net SD_DAT2: track 0.00 -> 7.55 mm, vias 0 -> 2
- net IMU2_INT4: track 0.00 -> 4.62 mm
- net Net-(SD1-CLK): track 0.00 -> 3.91 mm
- net IMU2_CSB1: track 8.04 -> 4.18 mm
- net SPI4_MISO: track 21.1 -> 17.4 mm
- net GND: track 0.00 -> 3.65 mm, vias 0 -> 2
- net SPI2_IMU_MISO: track 4.86 -> 6.26 mm
- net INT2_IMU: track 5.44 -> 6.27 mm
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Other:
- board size 45 x 45 mm -> 40 x 40 mm

Commit message: 10-04-2026
Parts:
- C12, C15, C16, C20, C23, C24, C26, C3, C30, C4, C5, C6, C7, C8, FB1, R13, U8: moved to B.Cu
- moved C3 116.0 mm to (133.6, 81.1), turned to 180 degrees
- moved C20 108.3 mm to (133.3, 82.3)
- moved C26 106.1 mm to (131.4, 83.5), turned to -90 degrees
- moved C4 105.0 mm to (118.1, 86.2), turned to 90 degrees
- moved C2 104.4 mm to (124.2, 72.2)
- moved C8 104.2 mm to (129.9, 65.0), turned to 90 degrees
- moved C1 104.0 mm to (127.1, 64.5), turned to -90 degrees
- moved C23 103.5 mm to (133.9, 68.9), turned to 90 degrees
- moved C7 100.7 mm to (128.7, 65.0), turned to 90 degrees
- moved C30 100.4 mm to (116.8, 89.5), turned to 180 degrees
- moved C16 99.0 mm to (115.2, 83.3), turned to 135 degrees
- moved R12 97.6 mm to (120.9, 91.7)
- moved R1 97.1 mm to (128.7, 64.5), turned to -90 degrees
- moved R10 96.1 mm to (118.7, 88.1)
- moved C12 95.7 mm to (125.9, 61.9), turned to -90 degrees
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Connections:
- C4 pad 2: Net-(C3-Pad2) -> Net-(C4-Pad2)
- U2 pad 16: unconnected-(U2-PC1-Pad16) -> IMU2_CSB1
- U2 pad 17: unconnected-(U2-PC2_C-Pad17) -> IMU2_INT3
- U2 pad 3: IMU2_CSB1 -> unconnected-(U2-PE4-Pad3)
- U2 pad 73: Net-(C3-Pad2) -> Net-(C4-Pad2)
- U2 pad 98: IMU2_INT3 -> unconnected-(U2-PE1-Pad98)
Routing:
- net +3.3V: track 0.00 -> 7.66 mm
- net SPI4_MISO: track 17.4 -> 22.2 mm
- net GND: track 3.65 -> 7.68 mm, vias 2 -> 6
- net IMU2_INT3: track 6.28 -> 2.26 mm, vias 2 -> 1
- net IMU2_CSB1: track 4.18 -> 0.96 mm, vias 2 -> 1
- net IMU2_INT2: track 2.47 -> 0.00 mm
- net IMU2_INT1: track 4.23 -> 2.09 mm, vias 2 -> 1
- net SD_CLK: track 11.1 -> 13.2 mm
- net Net-(SD1-CLK): track 3.91 -> 2.38 mm
- net IMU2_CSB2: track 5.06 -> 3.98 mm
- net IMU2_INT4: track 4.62 -> 3.63 mm, vias 0 -> 1
- net SPI4_MOSI: track 7.68 -> 8.28 mm, vias 3 -> 1
- net SPI4_SCLK: track 10.5 -> 11.0 mm, vias 3 -> 2

Commit message: 15-04-2026
Parts:
- added H1: MountingHole, MountingHole:MountingHole_2.7mm_M2.5_DIN965, F.Cu at (107.3, 68.3)
- added H2: MountingHole, MountingHole:MountingHole_2.7mm_M2.5_DIN965, F.Cu at (131.8, 92.8)
- moved R4 108.1 mm to (138.3, 72.0), turned to 90 degrees
- moved R5 106.0 mm to (136.9, 72.0), turned to 90 degrees
- moved D1 103.5 mm to (138.4, 74.4), turned to -90 degrees
- moved D2 101.5 mm to (136.9, 74.4), turned to -90 degrees
- moved U1 7.45 mm to (106.9, 77.2)
- moved U8 3.46 mm to (132.4, 87.5)
- moved Y1 0.46 mm to (122.0, 61.2), turned to -135 degrees
Routing:
- net LED0: track 0.00 -> 8.32 mm, vias 0 -> 1
- net LED1: track 0.00 -> 6.14 mm, vias 0 -> 1
- net Net-(D1-K): track 0.00 -> 1.44 mm
- net Net-(D2-K): track 0.00 -> 1.42 mm

Commit message: 23-04-2026
Parts:
- added FPC1: AFC24-S40FIA-HF, New_Library:FPC-SMD_40P-P0.50_AFC24-S40FIA-HF, B.Cu at (137.3, 77.9)
- moved R4 3.48 mm to (139.5, 68.7)
- moved R5 3.48 mm to (138.1, 68.8)
- moved D1 3.48 mm to (139.6, 71.2)
- moved D2 3.48 mm to (138.1, 71.2)
- moved C13 1.11 mm to (125.3, 82.8), turned to 180 degrees
- moved C23 0.94 mm to (133.2, 68.2)
Connections:
- U2 pad 32: unconnected-(U2-PC4-Pad32) -> ADC
- U2 pad 39: unconnected-(U2-PE9-Pad39) -> MOTOR1
- U2 pad 41: unconnected-(U2-PE11-Pad41) -> MOTOR2
- U2 pad 43: unconnected-(U2-PE13-Pad43) -> MOTOR3
- U2 pad 44: unconnected-(U2-PE14-Pad44) -> MOTOR4
- U2 pad 46: unconnected-(U2-PB10-Pad46) -> I2C2_SCL
- U2 pad 47: unconnected-(U2-PB11-Pad47) -> I2C2_SDA
- U2 pad 55: SPI2_IMU_CS -> UART2_TX
- U2 pad 56: unconnected-(U2-PD9-Pad56) -> UART2_RX
- U2 pad 57: unconnected-(U2-PD10-Pad57) -> SPI2_IMU_CS
- U2 pad 58: unconnected-(U2-PD11-Pad58) -> MOTOR5
- U2 pad 59: unconnected-(U2-PD12-Pad59) -> MOTOR6
- U2 pad 61: unconnected-(U2-PD14-Pad61) -> MOTOR7
- U2 pad 62: unconnected-(U2-PD15-Pad62) -> MOTOR8
- U2 pad 63: unconnected-(U2-PC6-Pad63) -> USART6_TX
- U2 pad 64: unconnected-(U2-PC7-Pad64) -> USART6_RX
- U2 pad 68: unconnected-(U2-PA9-Pad68) -> USART1_TX
- U2 pad 69: unconnected-(U2-PA10-Pad69) -> USART1_RX
- U2 pad 70: unconnected-(U2-PA11-Pad70) -> USB_D-
- U2 pad 71: unconnected-(U2-PA12-Pad71) -> USB_D+
Routing:
- net CAN_L: track 0.00 -> 40.7 mm, vias 0 -> 2
- net CAN_H: track 0.00 -> 38.2 mm, vias 0 -> 2
- net SDA_BARO: track 12.7 -> 43.7 mm, vias 2 -> 3
- net SCL_BARO: track 11.8 -> 40.9 mm, vias 2 -> 3
- net USART1_RX: track 0.00 -> 29.0 mm, vias 0 -> 2
- net USB_D-: track 0.00 -> 28.8 mm, vias 0 -> 2
- net I2C2_SDA: track 0.00 -> 26.7 mm, vias 0 -> 2
- net USB_D+: track 0.00 -> 25.4 mm, vias 0 -> 2
- net USART1_TX: track 0.00 -> 25.1 mm, vias 0 -> 2
- net I2C2_SCL: track 0.00 -> 19.8 mm, vias 0 -> 2
- net LED0: track 8.32 -> 0.00 mm, vias 1 -> 0
- net LED1: track 6.14 -> 0.01 mm, vias 1 -> 0
- net UART2_RX: track 0.00 -> 2.53 mm, vias 0 -> 1
- net UART2_TX: track 0.00 -> 2.38 mm, vias 0 -> 1
- net SD_CLK: track 13.2 -> 11.5 mm, vias 2 -> 1
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
Commit message: 24-04-2026
Parts:
- moved C20 0.71 mm to (133.2, 83.0)
- moved C3 0.71 mm to (133.5, 81.8)
- moved C21 0.45 mm to (124.1, 80.4)
- moved C18 0.45 mm to (121.5, 80.4)
- moved FB3 0.45 mm to (122.8, 80.4)
Routing:
- net USART6_RX: track 0.00 -> 24.8 mm, vias 0 -> 2
- net USART6_TX: track 0.00 -> 17.8 mm, vias 0 -> 2
- net ADC: track 0.00 -> 17.8 mm, vias 0 -> 2
- net UART2_RX: track 2.53 -> 18.0 mm, vias 1 -> 2
- net UART2_TX: track 2.38 -> 12.2 mm, vias 1 -> 2
- net USART1_TX: track 25.1 -> 27.4 mm
- net USART1_RX: track 29.0 -> 29.9 mm

Commit message: 28-04-2026
Parts:
- moved U8 25.4 mm to (133.9, 62.2)
- moved C11 24.2 mm to (136.9, 63.6), turned to 0 degrees
- moved C13 23.0 mm to (131.2, 60.6), turned to 90 degrees
- moved C20 22.7 mm to (136.8, 60.5)
- moved U3 22.5 mm to (134.0, 62.2)
- moved C26 22.0 mm to (136.3, 62.1)
- moved C3 3.83 mm to (131.1, 84.8), turned to 0 degrees
- moved C23 2.71 mm to (130.8, 66.9)
- moved C1 1.50 mm to (127.4, 63.1)
- moved FB1 1.50 mm to (127.5, 63.2)
- moved C8 1.50 mm to (130.2, 63.6)
- moved C7 1.50 mm to (129.0, 63.5)
- moved R1 1.50 mm to (129.0, 63.0)
Connections:
- U2 pad 23: unconnected-(U2-PA1-Pad23) -> RX_PPM
- U2 pad 35: unconnected-(U2-PB1-Pad35) -> BUZZER
Routing:
- net RX_PPM: track 0.00 -> 32.8 mm, vias 0 -> 2
- net +5V: track 0.00 -> 31.7 mm, vias 0 -> 5
- net BOOT: track 0.00 -> 20.6 mm, vias 0 -> 2
- net LED0: track 0.00 -> 19.3 mm, vias 0 -> 2
- net MOTOR6: track 0.00 -> 17.2 mm, vias 0 -> 2
- net BUZZER: track 0.00 -> 16.2 mm, vias 0 -> 2
- net MOTOR8: track 0.00 -> 16.2 mm, vias 0 -> 2
- net MOTOR1: track 0.00 -> 15.9 mm, vias 0 -> 2
- net MOTOR2: track 0.00 -> 15.7 mm, vias 0 -> 2
- net MOTOR7: track 0.00 -> 15.4 mm, vias 0 -> 2
- net MOTOR5: track 0.00 -> 15.0 mm, vias 0 -> 2
- net MOTOR4: track 0.00 -> 10.3 mm
- net MOTOR3: track 0.00 -> 10.3 mm
- net LED1: track 0.01 -> 9.81 mm, vias 0 -> 1
- net I2C2_SDA: track 26.7 -> 33.4 mm
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- added copper zone on In4.Cu, net +3.3V
- added copper zone on In6.Cu, net +3.3VA
- added copper zone on In6.Cu, net GND
