File: Vaimanika_H7_Sensor/Vaimanika_H7_Sensor.kicad_pcb (KiCad board)
At the start: 8 copper layers, 40 x 40 mm, 72 parts, among them SW1 TS-1088-AR02016, U1 TCAN334G, U2 STM32H743VITx, U3 NCP163ASN330T1G, U4 MS5611-01BA, U5 ICM-42688-P, U6 ICM-42688-P, U7 W25Q128JVS, U8 RT9080-33GJ5, U9 BMI088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

Commit message: 29-04-2026
Parts:
- moved C2 4.27 mm to (126.1, 68.3), turned to 90 degrees
- moved R3 3.07 mm to (110.1, 80.3), turned to 90 degrees
- moved C1 2.46 mm to (126.3, 65.2)
- moved FB1 2.46 mm to (127.3, 60.8)
- moved C24 1.58 mm to (119.3, 62.8)
- moved C8 1.53 mm to (128.8, 64.1), turned to 0 degrees
- moved C23 1.04 mm to (131.1, 67.9)
- moved C13 1.00 mm to (131.8, 59.8)
- moved C26 0.94 mm to (136.3, 63.0)
- moved C20 0.88 mm to (137.4, 59.9), turned to 45 degrees
- moved C22 0.87 mm to (131.3, 74.7), turned to 180 degrees
- moved C3 0.84 mm to (131.9, 84.8), turned to 90 degrees
- moved C19 0.78 mm to (134.9, 74.7), turned to 0 degrees
- moved C7 0.69 mm to (128.5, 63.0), turned to 0 degrees
- moved C11 0.60 mm to (137.0, 63.0)
Routing:
- net +3.3VA: track 3.26 -> 51.9 mm, vias 1 -> 10
- net +3.3V: track 10.9 -> 47.3 mm, vias 0 -> 10
- net VDDA: track 0.00 -> 21.0 mm, vias 0 -> 3
- net GND: track 10.4 -> 18.2 mm, vias 47 -> 48
- net HSE_O: track 0.00 -> 7.74 mm
- net HSE_I: track 0.00 -> 7.53 mm
- net Net-(C3-Pad2): track 0.00 -> 4.60 mm
- net Net-(U5-VDD): track 0.00 -> 4.54 mm
- net SPI1_IMU_MOSI: track 6.46 -> 10.9 mm
- net Net-(U6-VDD): track 0.00 -> 4.16 mm
- net SPI4_MISO: track 22.2 -> 26.2 mm
- net Net-(U9-VDDIO): track 0.00 -> 3.98 mm
- net SPI1_IMU_MISO: track 6.71 -> 10.7 mm
- net SCL_BARO: track 40.8 -> 43.8 mm
- net SPI1_IMU_SCLK: track 8.80 -> 11.9 mm
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
Commit message: 01-05-2026
Parts:
- C12, C24, C26: moved to F.Cu
- C17, C27, C28: moved to B.Cu
- moved C17 105.6 mm to (136.9, 63.9)
- moved C27 99.8 mm to (137.6, 59.8), turned to 45 degrees
- moved C28 99.5 mm to (136.9, 62.7)
- moved TP1 53.9 mm to (130.6, 71.0)
- moved TP2 47.3 mm to (126.7, 61.5)
- moved C20 27.6 mm to (130.3, 86.6), turned to 180 degrees
- moved C26 18.5 mm to (120.5, 72.7), turned to 180 degrees
- moved C24 11.9 mm to (124.7, 73.4), turned to 45 degrees
- moved U1 6.25 mm to (110.7, 72.3)
- moved C12 4.60 mm to (121.4, 60.8), turned to 0 degrees
- moved C6 4.16 mm to (110.7, 76.2), turned to 90 degrees
- moved C5 1.26 mm to (109.7, 74.7), turned to 0 degrees
- moved Y1 0.73 mm to (121.2, 61.1)
Connections:
- FPC1 pad 16: GND -> unconnected-(FPC1-Pad16)
Routing:
- net +3.3V: track 47.3 -> 97.5 mm, vias 10 -> 20
- net RST: track 0.00 -> 31.3 mm, vias 0 -> 2
- net IMU2_CSB1: track 0.96 -> 10.2 mm, vias 1 -> 2
- net SD_CLK: track 11.5 -> 19.8 mm, vias 1 -> 2
- net IMU2_INT3: track 2.26 -> 10.0 mm
- net IMU2_INT2: track 0.00 -> 7.56 mm
- net IMU2_INT1: track 2.09 -> 9.02 mm
- net GND: track 18.2 -> 23.8 mm, vias 48 -> 50
- net SD_CD: track 0.00 -> 5.42 mm
- net IMU2_CSB2: track 3.98 -> 8.27 mm
- net CAN_RXD: track 0.00 -> 4.05 mm
- net CAN_TXD: track 0.00 -> 3.73 mm
- net IMU2_INT4: track 3.63 -> 6.49 mm, vias 1 -> 0
- net CAN_H: track 38.2 -> 35.7 mm
- net Net-(C4-Pad2): track 0.00 -> 2.32 mm
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Other:
- board text added: "Put that thing back"

Commit message: 18-05-2026
Parts:
- moved R4 34.7 mm to (107.2, 81.2), turned to -90 degrees
- moved D1 33.3 mm to (107.2, 78.8), turned to 90 degrees
- moved R5 31.9 mm to (108.6, 81.2), turned to -90 degrees
- moved D2 30.4 mm to (108.7, 78.8), turned to 90 degrees
Connections:
- net UART2_RX renamed USART3_RX
- net UART2_TX renamed USART3_TX
- U2 pad 37: LED1 -> UART7_RX
- U2 pad 38: LED0 -> UART7_TX
- U2 pad 81: unconnected-(U2-PD0-Pad81) -> UART4_RX
- U2 pad 82: unconnected-(U2-PD1-Pad82) -> UART4_TX
- U2 pad 86: unconnected-(U2-PD5-Pad86) -> USART2_TX
- U2 pad 87: unconnected-(U2-PD6-Pad87) -> USART2_RX
Routing:
- net LED0: track 19.3 -> 0.01 mm, vias 2 -> 0
- net LED1: track 9.81 -> 0.00 mm, vias 1 -> 0
- net UART7_TX: track 0.00 -> 9.15 mm, vias 0 -> 1
- net UART7_RX: track 0.00 -> 4.80 mm, vias 0 -> 1
- net GND: vias 50 -> 49

Commit message: 20-05-2026
Parts:
- added U10: WAFER-GH1.25-4PWB, New_Library:CONN-SMD_4P-P1.25_XUNPU_WAFER-GH1.25-4PWB, F.Cu at (106.7, 92.1)
- added U11: WAFER-GH1.25-4PWB, New_Library:CONN-SMD_4P-P1.25_XUNPU_WAFER-GH1.25-4PWB, F.Cu at (106.5, 62.5)
- added U12: WAFER-GH1.25-4PWB, New_Library:CONN-SMD_4P-P1.25_XUNPU_WAFER-GH1.25-4PWB, F.Cu at (138.5, 68.0)
- added U13: WAFER-GH1.25-4PWB, New_Library:CONN-SMD_4P-P1.25_XUNPU_WAFER-GH1.25-4PWB, F.Cu at (138.4, 92.5)
- moved G*** 16.4 mm to (123.9, 94.9)
- moved C6 1.10 mm to (109.7, 75.8), turned to 0 degrees
- renumbered TP3 to SD_CD
Connections:
- U2 pad 3: unconnected-(U2-PE4-Pad3) -> IMU2_CSB2
- U2 pad 97: IMU2_CSB2 -> UART8_RX
- U2 pad 98: unconnected-(U2-PE1-Pad98) -> UART8_TX
Routing:
- net +5V: track 36.1 -> 139.8 mm, vias 5 -> 9
- net UART8_TX: track 0.00 -> 46.5 mm, vias 0 -> 2
- net UART8_RX: track 0.00 -> 42.9 mm, vias 0 -> 2
- net UART4_RX: track 0.00 -> 28.8 mm, vias 0 -> 2
- net UART4_TX: track 0.00 -> 28.1 mm, vias 0 -> 2
- net USART2_RX: track 0.00 -> 24.6 mm, vias 0 -> 2
- net USART2_TX: track 0.00 -> 24.5 mm, vias 0 -> 2
- net UART7_RX: track 4.80 -> 12.5 mm
- net IMU2_CSB1: track 10.2 -> 13.3 mm
- net UART7_TX: track 9.15 -> 12.2 mm
- net GND: track 23.8 -> 26.1 mm, vias 49 -> 50
- net IMU2_CSB2: track 8.27 -> 7.78 mm, vias 2 -> 1
Other:
- board text added: "UART2"
- board text added: "UART4"
- board text added: "UART7"
- board text added: "UART8"

Commit message: 20-05-2026
Parts:
- added G***: LOGO, LOGO, F.Cu at (113.6, 94.7)
- moved G*** 38.0 mm to (140.1, 60.5)
- moved SD_CD 2.30 mm to (109.2, 82.3)
- moved C12 0.94 mm to (121.3, 59.9)
- renumbered TP1 to INT_2, TP2 to INT_4
Routing:
- net IMU2_CSB1: track 13.3 -> 4.04 mm, vias 2 -> 1
- net SD_CMD: track 16.4 -> 23.4 mm
- net GND: track 26.1 -> 32.4 mm, vias 50 -> 58
- net SD_CLK: track 19.8 -> 24.7 mm
- net SD_DAT3: track 11.8 -> 15.0 mm
- net CS_FLASH: track 12.0 -> 15.0 mm, vias 1 -> 2
- net SD_DAT2: track 9.98 -> 12.6 mm
- net +3.3V: track 97.5 -> 98.1 mm
- net SD_CD: track 5.42 -> 5.98 mm
- net HSE_O: track 7.33 -> 7.83 mm
Other:
- board text added: "AEROSPACE"
- board text added: "Designed in Bihar."
- board text added: "Manufactured in India."
- board text added: "VAIMANIKA"

Commit message: 20-05-2026
Routing:
- net VDDA: track 21.0 -> 21.5 mm
- net GND: vias 58 -> 59
- added copper zone on In3.Cu, net GND
Changed lines of the file:
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@@
 	)
 	(via
-		(at 103.38 88.61)
+		(at 103.38 89.51)
 		(size 0.6)
 		(drill 0.3)
@@
 	)
 	(via
+		(at 125.75 80.17)
+		(size 0.6)
+		(drill 0.3)
+		(layers "F.Cu" "B.Cu")
+		(free yes)
+		(net 1)
+	)
+	(via
 		(at 120.02 65.69)
 		(size 0.8)
@@
 	)
 	(segment
+		(start 126.65 68)
+		(end 127.150001 68)
+		(width 0.3)
+		(layer "B.Cu")
+		(net 2)
+	)
+	(segment
 		(start 127.44 63.63)
 		(end 126.12 63.63)
@@
 			)
 		)
+	)
+	(zone
+		(net 1)
+		(net_name "GND")
+		(layer "In3.Cu")
+		(hatch edge 0.5)
+		(priority 6)
+		(connect_pads
+			(clearance 0.3)
+		)
+		(min_thickness 0.25)
+		(filled_areas_thickness no)
+		(fill yes
+			(thermal_gap 0.5)
+			(thermal_bridge_width 0.5)
+		)
+		(polygon
+			(pts
+				(xy 99.95 56.42) (xy 144.3 56.42) (xy 145.1 57.22) (xy 145.1 99.46) (xy 99.95 99.46)
+			)
+		)

Commit message: 21-05-2026
Parts:
- moved G*** 2.23 mm to (115.8, 94.6)
Other:
- board text added: "VA-VEG_H7-FC-S-R01"

Commit message: 22-05-2026
Parts:
- added G***: LOGO, LOGO, F.Cu at (158.1, 93.4)
- added G***: LOGO, LOGO, F.Cu at (127.7, 85.2)
- added G***: LOGO, LOGO, F.Cu at (165.0, 81.4)
- added G***: LOGO, LOGO, F.Cu at (155.0, 100.5)
Routing:
- net GND: track 32.4 -> 35.0 mm, vias 59 -> 60
