File: Vaimanika_H7_Sensor/Vaimanika_H7_Sensor.kicad_pcb (KiCad board)
At the start: 8 copper layers, 40 x 40 mm, 81 parts, among them SW1 TS-1088-AR02016, U1 TCAN334G, U10 WAFER-GH1.25-4PWB, U11 WAFER-GH1.25-4PWB, U12 WAFER-GH1.25-4PWB, U13 WAFER-GH1.25-4PWB, U2 STM32H743VITx, U3 NCP163ASN330T1G, U4 MS5611-01BA, U5 ICM-42688-P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

Commit message: 25-05-2026
Parts:
- removed the G*** at (158.1, 93.4)
- removed the G*** at (165.0, 81.4)
- removed the G*** at (155.0, 100.5)
- added TP4: TestPoint, TestPoint:TestPoint_Pad_D1.0mm, B.Cu at (106.9, 82.3)
- added TP5: TestPoint, TestPoint:TestPoint_Pad_D1.0mm, B.Cu at (106.9, 80.2)
- renumbered INT_2 to TP1, INT_4 to TP2, SD_CD to TP3
Connections:
- U2 pad 77: unconnected-(U2-PA15-Pad77) -> PA15
Routing:
- net SD_DAT2: track 12.6 -> 23.4 mm
- net PA15: track 0.00 -> 8.98 mm
- net SD_DAT3: track 15.0 -> 23.7 mm
- net SD_DAT1: track 18.2 -> 24.3 mm
- net SD_DAT0: track 18.0 -> 24.0 mm
- net SD_CLK: track 24.7 -> 20.0 mm
- net USART2_RX: track 24.6 -> 27.3 mm
- net SD_CMD: track 23.4 -> 24.5 mm
- net INT2_IMU: track 7.26 -> 8.32 mm
- net SPI4_MOSI: track 8.28 -> 9.28 mm
- net SPI2_IMU_MOSI: track 8.59 -> 9.56 mm
- net SPI1_IMU_MOSI: track 10.9 -> 11.8 mm
- net SPI2_IMU_MISO: track 7.00 -> 7.83 mm
