File: Vaimanika_H7_Sensor/Vaimanika_H7_Sensor.kicad_sch (KiCad schematic)
At the start: 67 parts, among them SW1 TS-1088-AR02016, U1 TCAN334G, U2 STM32H743VITx, U3 NCP163ASN330T1G, U4 MS5611-01BA, U5 ICM-42688-P, U6 ICM-42688-P, U7 W25Q128JVS, U8 RT9080-33GJ5, U9 BMI088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

Commit message: 12-03-2026-02nd
Connections:
- net IMU2_INT1: now also U2.15 (PC0); no longer U2.35 (PB1)
Changed lines of the file:
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@@
 	(global_label "IMU2_INT1"
 		(shape input)
-		(at 104.14 96.52 0)
+		(at 104.14 137.16 0)
 		(fields_autoplaced yes)
 		(effects
@@
 		)
 		(property "Intersheetrefs" "${INTERSHEET_REFS}"
-			(at 116.8014 96.52 0)
+			(at 116.8014 137.16 0)
 			(effects
 				(font

Commit message: 28-03-2025
Parts:
- removed TF1: TF-CARD H1.8, New_Library:TF-SMD_TF-CARD-H1.8, symbol New_Library:TF-CARDH1.8
- added SD1: TF-027-H300, New_Library:TF-SMD_HYCW104-TF08-375B, symbol New_Library:TF-027-H300
- added TP3: TestPoint, TestPoint:TestPoint_Pad_D1.0mm, symbol Connector:TestPoint
Connections:
- net +3.3V: now also SD1.4 (VDD)
- net GND: now also SD1.10, SD1.11, SD1.6 (VSS)
- net SD_CD: now also SD1.9, TP3.1; no longer U2.7 (PC13)
- net SD_CMD: now also SD1.3 (CMD)
- net SD_DAT0: now also SD1.7 (DAT0)
- net SD_DAT1: now also SD1.8 (DAT1)
- net SD_DAT2: now also SD1.1 (DAT2)
- net SD_DAT3: now also SD1.2 (CD/DAT3)
- net at R9.1: now also SD1.5 (CLK)

Commit message: 10-04-2026
Connections:
- net IMU2_CSB1: now also U2.16 (PC1); no longer U2.3 (PE4)
- net IMU2_INT3: now also U2.17 (PC2_C); no longer U2.98 (PE1)
- net at C3.2, U2.48 (VCAP): no longer C4.2, U2.73 (VCAP)
- new net: C4.2, U2.73 (VCAP)
Other:
- moved on the sheet: C3, C4
Changed lines of the file:
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@@
 	)
 	(junction
-		(at 58.42 162.56)
-		(diameter 0)
-		(color 0 0 0 0)
-	)
-	(junction
 		(at 49.53 60.96)
 		(diameter 0)
@@
 	)
 	(junction
-		(at 58.42 160.02)
-		(diameter 0)
-		(color 0 0 0 0)
-	)
-	(junction
 		(at 83.82 40.64)
 		(diameter 0)
@@
 	(wire
 		(pts
-			(xy 50.8 160.02) (xy 50.8 161.29)
+			(xy 50.8 157.48) (xy 50.8 161.29)
 		)
 		(stroke
@@
 	(wire
 		(pts
+			(xy 58.42 162.56) (xy 58.42 165.1)
+		)
+		(stroke
+			(width 0)
+			(type default)
+		)
+	)
+	(wire
+		(pts
 			(xy 259.08 44.45) (xy 262.89 44.45)
 		)
@@
 	(wire
 		(pts
-			(xy 58.42 160.02) (xy 58.42 162.56)
-		)
-		(stroke
-			(width 0)
-			(type default)
-		)
-	)
-	(wire
-		(pts
 			(xy 210.82 189.23) (xy 210.82 191.77)
 		)
@@
 	(wire
 		(pts
-			(xy 50.8 161.29) (xy 50.8 162.56)
+			(xy 50.8 161.29) (xy 50.8 165.1)
 		)
 		(stroke
@@
 		)
 	)
+	(wire
+		(pts
+			(xy 58.42 157.48) (xy 58.42 160.02)
+		)
+		(stroke
+			(width 0)
+			(type default)
+		)
+	)
 	(global_label "CS_FLASH"
 		(shape input)
@@
 	(global_label "IMU2_CSB1"
 		(shape input)
-		(at 58.42 83.82 180)
+		(at 104.14 139.7 0)
 		(fields_autoplaced yes)
 		(effects
@@
 				(size 1.27 1.27)
 			)
-			(justify right)
+			(justify left)
 		)
 		(property "Intersheetrefs" "${INTERSHEET_REFS}"
-			(at 44.912 83.82 0)
+			(at 117.648 139.7 0)
 			(effects
 				(font
 					(size 1.27 1.27)
 				)
-				(justify right)
+				(justify left)
 				(hide yes)
 			)
@@
 	(global_label "IMU2_INT3"
 		(shape input)
-		(at 58.42 76.2 180)
+		(at 104.14 142.24 0)
 		(fields_autoplaced yes)
 		(effects
@@
 				(size 1.27 1.27)
 			)
-			(justify right)
+			(justify left)
 		)
 		(property "Intersheetrefs" "${INTERSHEET_REFS}"
-			(at 45.7586 76.2 0)
+			(at 116.8014 142.24 0)
 			(effects
 				(font
 					(size 1.27 1.27)
 				)
-				(justify right)
+				(justify left)
 				(hide yes)
 			)
@@
 	(symbol
 		(lib_id "Device:C")
-		(at 54.61 160.02 90)
+		(at 54.61 157.48 90)
 		(unit 1)
 		(exclude_from_sim no)
@@
 		(dnp no)
 		(property "Reference" "C3"
-			(at 54.61 153.416 90)
+			(at 54.61 150.876 90)
 			(effects
 				(font
@@
 		)
 		(property "Value" "2.2uF"
-			(at 54.61 155.956 90)
+			(at 54.61 153.416 90)
 			(effects
 				(font
@@
 		)
 		(property "Footprint" "Capacitor_SMD:C_0402_1005Metric"
-			(at 58.42 159.0548 0)
+			(at 58.42 156.5148 0)
 			(effects
 				(font
@@
 		)
 		(property "Datasheet" "~"
-			(at 54.61 160.02 0)
+			(at 54.61 157.48 0)
 			(effects
 				(font
@@
 		)
 		(property "Description" "Unpolarized capacitor"
-			(at 54.61 160.02 0)
+			(at 54.61 157.48 0)
 			(effects
 				(font
@@
 		)
 		(property "LCSC" "C20539421"
-			(at 54.61 160.02 90)
+			(at 54.61 157.48 90)
 			(effects
 				(font
@@
 		)
 		(property "BOARD" "SENSOR"
-			(at 54.61 160.02 90)
+			(at 54.61 157.48 90)
 			(effects
 				(font
@@
 	(symbol
 		(lib_id "Device:C")
-		(at 54.61 162.56 90)
+		(at 54.61 165.1 90)
 		(unit 1)
 		(exclude_from_sim no)
@@
 		(dnp no)
 		(property "Reference" "C4"
-			(at 54.61 168.402 90)
+			(at 54.61 170.942 90)
 			(effects
 				(font
@@
 		)
 		(property "Value" "2.2uF"
-			(at 54.61 166.116 90)
+			(at 54.61 168.656 90)
 			(effects
 				(font
@@
 		)
 		(property "Footprint" "Capacitor_SMD:C_0402_1005Metric"
-			(at 58.42 161.5948 0)
+			(at 58.42 164.1348 0)
 			(effects
 				(font
@@
 		)
 		(property "Datasheet" "~"
-			(at 54.61 162.56 0)
+			(at 54.61 165.1 0)
 			(effects
 				(font
@@
 		)
 		(property "Description" "Unpolarized capacitor"
-			(at 54.61 162.56 0)
+			(at 54.61 165.1 0)
 			(effects
 				(font
@@
 		)
 		(property "LCSC" "C20539421"
-			(at 54.61 162.56 90)
+			(at 54.61 165.1 90)
 			(effects
 				(font
@@
 		)
 		(property "BOARD" "SENSOR"
-			(at 54.61 162.56 90)
+			(at 54.61 165.1 90)
 			(effects
 				(font

Commit message: 15-04-2026
Parts:
- added H1, H2: MountingHole, MountingHole:MountingHole_2.7mm_M2.5_DIN965, symbol Mechanical:MountingHole
- added J1: Conn_01x08_Socket, symbol Connector:Conn_01x08_Socket
Changed lines of the file:
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@@
 	(text_box ""
 		(exclude_from_sim no)
+		(at 233.68 175.26 0)
+		(size 99.06 55.88)
+		(margins 0.9525 0.9525 0.9525 0.9525)
+		(stroke
+			(width 0)
+			(type solid)
+		)
+		(fill
+			(type none)
+		)
+		(effects
+			(font
+				(size 1.27 1.27)
+			)
+			(justify right top)
+		)
+	)
+	(text_box ""
+		(exclude_from_sim no)
 		(at 170.18 121.92 0)
 		(size 54.61 29.21)
@@
 	)
 	(symbol
+		(lib_id "Mechanical:MountingHole")
+		(at 308.61 180.34 0)
+		(unit 1)
+		(exclude_from_sim no)
+		(in_bom no)
+		(on_board yes)
+		(dnp no)
+		(fields_autoplaced yes)
+		(property "Reference" "H1"
+			(at 311.15 179.0699 0)
+			(effects
+				(font
+					(size 1.27 1.27)
+				)
+				(justify left)
+			)
+		)
+		(property "Value" "MountingHole"
+			(at 311.15 181.6099 0)
+			(effects
+				(font
+					(size 1.27 1.27)
+				)
+				(justify left)
+			)
+		)
+		(property "Footprint" "MountingHole:MountingHole_2.7mm_M2.5_DIN965"
+			(at 308.61 180.34 0)
+			(effects
+				(font
+					(size 1.27 1.27)
+				)
+				(hide yes)
+			)
+		)
+		(property "Datasheet" "~"
+			(at 308.61 180.34 0)
+			(effects
+				(font
+					(size 1.27 1.27)
+				)
+				(hide yes)
+			)
+		)
+		(property "Description" "Mounting Hole without connection"
+			(at 308.61 180.34 0)
+			(effects
+				(font
+					(size 1.27 1.27)
+				)
+				(hide yes)
+			)
+		)
+		(instances
+			(project ""
+				(path "/23770a09-842c-46e7-8c45-82f07b31c15d"
+					(reference "H1")
+					(unit 1)
+				)
+			)
+		)
+	)
+	(symbol
 		(lib_id "Device:R")
 		(at 261.62 132.08 180)
@@
 	)
 	(symbol
+		(lib_id "Mechanical:MountingHole")
+		(at 308.61 185.42 0)
+		(unit 1)
+		(exclude_from_sim no)
+		(in_bom no)
+		(on_board yes)
+		(dnp no)
+		(fields_autoplaced yes)
+		(property "Reference" "H2"
+			(at 311.15 184.1499 0)
+			(effects
+				(font
+					(size 1.27 1.27)
+				)
+				(justify left)
+			)
+		)
+		(property "Value" "MountingHole"
+			(at 311.15 186.6899 0)
+			(effects
+				(font
+					(size 1.27 1.27)
+				)
+				(justify left)
+			)
+		)
+		(property "Footprint" "MountingHole:MountingHole_2.7mm_M2.5_DIN965"
+			(at 308.61 185.42 0)
+			(effects
+				(font
+					(size 1.27 1.27)
+				)
+				(hide yes)
+			)
+		)
+		(property "Datasheet" "~"
+			(at 308.61 185.42 0)
+			(effects
+				(font
+					(size 1.27 1.27)
+				)
+				(hide yes)
+			)
+		)
+		(property "Description" "Mounting Hole without connection"
+			(at 308.61 185.42 0)
+			(effects
+				(font
+					(size 1.27 1.27)
+				)
+				(hide yes)
+			)
+		)
+		(instances
+			(project "Vaimanika_H7_Sensor"
+				(path "/23770a09-842c-46e7-8c45-82f07b31c15d"
+					(reference "H2")
+					(unit 1)
+				)
+			)
+		)
+	)
+	(symbol
 		(lib_id "power:+3.3V")
 		(at 213.36 100.33 0)
@@
 					(unit 1)
 				)
+			)
+		)
+	)
+	(symbol
+		(lib_id "Connector:Conn_01x08_Socket")
+		(at 312.42 199.39 0)
+		(unit 1)
+		(exclude_from_sim no)
+		(in_bom yes)
+		(on_board yes)
+		(dnp no)
+		(fields_autoplaced yes)
+		(property "Reference" "J1"
+			(at 313.69 199.3899 0)
+			(effects
+				(font
+					(size 1.27 1.27)
+				)
+				(justify left)
+			)
+		)
+		(property "Value" "Conn_01x08_Socket"
+			(at 313.69 201.9299 0)
+			(effects
+				(font
+					(size 1.27 1.27)
+				)
+				(justify left)
+			)
+		)
+		(property "Footprint" ""
+			(at 312.42 199.39 0)
+			(effects
+				(font
+					(size 1.27 1.27)
+				)
+				(hide yes)
+			)
+		)
+		(property "Datasheet" "~"
+			(at 312.42 199.39 0)
+			(effects
+				(font
+					(size 1.27 1.27)
+				)
+				(hide yes)
+			)
+		)
+		(property "Description" "Generic connector, single row, 01x08, script generated"
+			(at 312.42 199.39 0)
+			(effects
+				(font
+					(size 1.27 1.27)
+				)
+				(hide yes)
+			)
+		)
+		(pin "3"
+		)
+		(pin "7"
+		)
+		(pin "1"
+		)
+		(pin "2"
+		)
+		(pin "5"
+		)
+		(pin "6"
+		)
+		(pin "4"
+		)
+		(pin "8"
+		)
+		(instances
+			(project ""
+				(path "/23770a09-842c-46e7-8c45-82f07b31c15d"
+					(reference "J1")
+					(unit 1)
+				)

Commit message: 23-04-2026
Parts:
- removed J1: Conn_01x08_Socket, symbol Connector:Conn_01x08_Socket
- added FPC1: AFC24-S40FIA-HF, New_Library:FPC-SMD_40P-P0.50_AFC24-S40FIA-HF, symbol New_Library:AFC24-S40FIA-HF
Connections:
- net +5V: now also FPC1.3, FPC1.4, FPC1.5, FPC1.6
- net CAN_H: now also FPC1.14
- net CAN_L: now also FPC1.15
- net GND: now also FPC1.1, FPC1.10, FPC1.13, FPC1.16, FPC1.2, FPC1.29, FPC1.41, FPC1.42, FPC1.7, FPC1.8, FPC1.9
- net SCL_BARO: now also FPC1.18
- net SDA_BARO: now also FPC1.17
- net SPI2_IMU_CS: now also U2.57 (PD10); no longer U2.55 (PD8)
- net ADC: now reaches U2.32 (PC4)
- net ADC: now also FPC1.30
- net MOTOR1: now reaches U2.39 (PE9)
- net MOTOR1: now also FPC1.33
- net MOTOR2: now reaches U2.41 (PE11)
- net MOTOR2: now also FPC1.34
- net MOTOR3: now reaches U2.43 (PE13)
- net MOTOR3: now also FPC1.35
- net MOTOR4: now reaches U2.44 (PE14)
- net MOTOR4: now also FPC1.36
- net I2C2_SCL: now reaches U2.46 (PB10)
- net I2C2_SCL: now also FPC1.19
- net I2C2_SDA: now reaches U2.47 (PB11)
- net I2C2_SDA: now also FPC1.20
- net UART2_RX: now reaches U2.56 (PD9)
- net UART2_RX: now also FPC1.26
- net MOTOR5: now reaches U2.58 (PD11)
- net MOTOR5: now also FPC1.37
- net MOTOR6: now reaches U2.59 (PD12)
- net MOTOR6: now also FPC1.38
- net MOTOR7: now reaches U2.61 (PD14)
- net MOTOR7: now also FPC1.39
- net MOTOR8: now reaches U2.62 (PD15)
- net MOTOR8: now also FPC1.40
- net USART6_TX: now reaches U2.63 (PC6)
- net USART6_TX: now also FPC1.27
- net USART6_RX: now reaches U2.64 (PC7)
- net USART6_RX: now also FPC1.28
- net USART1_TX: now reaches U2.68 (PA9)
- net USART1_TX: now also FPC1.21
- net USART1_RX: now reaches U2.69 (PA10)
- net USART1_RX: now also FPC1.22
- net USB_D-: now reaches U2.70 (PA11)
- net USB_D-: now also FPC1.12
- net USB_D+: now reaches U2.71 (PA12)
- net USB_D+: now also FPC1.11
- new net BUZZER: FPC1.32
- new net RX_PPM: FPC1.31
- new net UART2_TX: FPC1.25, U2.55 (PD8)
Other:
- note added: "Pin 7 and 8 are Empty could be sued for different purpose adn for now conencted to Gnd"
- moved on the sheet: C3, C4

Commit message: 28-04-2026
Connections:
- net BUZZER: now also U2.35 (PB1)
- net RX_PPM: now also U2.23 (PA1)
Changed lines of the file:
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@@
+		)
+	)
+	(global_label "BUZZER"
+		(shape input)
+		(at 104.14 96.52 0)
+		(fields_autoplaced yes)
+		(effects
+			(font
+				(size 1.27 1.27)
+			)
+			(justify left)
+		)
+		(property "Intersheetrefs" "${INTERSHEET_REFS}"
+			(at 114.5637 96.52 0)
+			(effects
+				(font
+					(size 1.27 1.27)
+				)
+				(justify left)
+				(hide yes)
+			)
 		)
 	)
@@
 				(hide yes)
 			)
+		)
+	)
+	(global_label "RX_PPM"
+		(shape input)
+		(at 104.14 53.34 0)
+		(fields_autoplaced yes)
+		(effects
+			(font
+				(size 1.27 1.27)
+			)
+			(justify left)
+		)
+		(property "Intersheetrefs" "${INTERSHEET_REFS}"
+			(at 114.5637 53.34 0)
+			(effects
+				(font
+					(size 1.27 1.27)
+				)
+				(justify left)
+				(hide yes)
+			)

Commit message: 01-05-2026
Connections:
- net GND: no longer FPC1.16
- net USART1_RX: now also U2.87 (PD6)
- net USART1_TX: now also U2.86 (PD5)
- net UART4_RX: now reaches U2.81 (PD0)
- net UART4_TX: now reaches U2.82 (PD1)
- net UART2_RX renamed USART3_RX
- net UART2_TX renamed USART3_TX
- no-connect marks 9 -> 10
Changed lines of the file:
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@@
 	)
 	(junction
-		(at 388.62 67.31)
-		(diameter 0)
-		(color 0 0 0 0)
-	)
-	(junction
 		(at 388.62 59.69)
 		(diameter 0)
@@
 	)
 	(no_connect
+		(at 389.89 67.31)
+	)
+	(no_connect
 		(at 158.75 213.36)
 	)
@@
 	(wire
 		(pts
-			(xy 389.89 67.31) (xy 388.62 67.31)
-		)
-		(stroke
-			(width 0)
-			(type default)
-		)
-	)
-	(wire
-		(pts
 			(xy 388.62 46.99) (xy 388.62 44.45)
 		)
@@
 	(wire
 		(pts
-			(xy 388.62 59.69) (xy 388.62 67.31)
+			(xy 388.62 59.69) (xy 388.62 100.33)
 		)
 		(stroke
@@
 	(wire
 		(pts
-			(xy 388.62 67.31) (xy 388.62 100.33)
-		)
-		(stroke
-			(width 0)
-			(type default)
-		)
-	)
-	(wire
-		(pts
 			(xy 144.78 72.39) (xy 144.78 74.93)
 		)
@@
 		)
 	)
-	(global_label "UART2_TX"
+	(global_label "USART3_TX"
 		(shape input)
 		(at 389.89 90.17 180)
@@
 		)
 		(property "Intersheetrefs" "${INTERSHEET_REFS}"
-			(at 377.8939 90.17 0)
+			(at 376.6844 90.17 0)
 			(effects
 				(font
@@
 		)
 	)
+	(global_label "UART4_TX"
+		(shape input)
+		(at 58.42 119.38 180)
+		(fields_autoplaced yes)
+		(effects
+			(font
+				(size 1.27 1.27)
+			)
+			(justify right)
+		)
+		(property "Intersheetrefs" "${INTERSHEET_REFS}"
+			(at 46.4239 119.38 0)
+			(effects
+				(font
+					(size 1.27 1.27)
+					(italic yes)
+				)
+				(justify right)
+				(hide yes)
+			)
+		)
+	)
 	(global_label "MOTOR8"
 		(shape input)
@@
 		)
 	)
+	(global_label "USART1_RX"
+		(shape input)
+		(at 58.42 132.08 180)
+		(fields_autoplaced yes)
+		(effects
+			(font
+				(size 1.27 1.27)
+			)
+			(justify right)
+		)
+		(property "Intersheetrefs" "${INTERSHEET_REFS}"
+			(at 44.912 132.08 0)
+			(effects
+				(font
+					(size 1.27 1.27)
+					(italic yes)
+				)
+				(justify right)
+				(hide yes)
+			)
+		)
+	)
 	(global_label "BUZZER"
 		(shape input)
@@
 		)
 	)
-	(global_label "UART2_RX"
+	(global_label "USART3_RX"
 		(shape input)
 		(at 58.42 139.7 180)
@@
 		)
 		(property "Intersheetrefs" "${INTERSHEET_REFS}"
-			(at 46.1215 139.7 0)
+			(at 44.912 139.7 0)
 			(effects
 				(font
@@
 		)
 	)
-	(global_label "UART2_TX"
+	(global_label "USART3_TX"
 		(shape input)
 		(at 58.42 137.16 180)
@@
 		)
 		(property "Intersheetrefs" "${INTERSHEET_REFS}"
-			(at 46.4239 137.16 0)
+			(at 45.2144 137.16 0)
 			(effects
 				(font
@@
 		)
 	)
-	(global_label "UART2_RX"
+	(global_label "USART3_RX"
 		(shape input)
 		(at 389.89 92.71 180)
@@
 		)
 		(property "Intersheetrefs" "${INTERSHEET_REFS}"
-			(at 377.5915 92.71 0)
+			(at 376.382 92.71 0)
 			(effects
 				(font
@@
 		)
 	)
+	(global_label "UART4_RX"
+		(shape input)
+		(at 58.42 116.84 180)
+		(fields_autoplaced yes)
+		(effects
+			(font
+				(size 1.27 1.27)
+			)
+			(justify right)
+		)
+		(property "Intersheetrefs" "${INTERSHEET_REFS}"
+			(at 46.1215 116.84 0)
+			(effects
+				(font
+					(size 1.27 1.27)
+					(italic yes)
+				)
+				(justify right)
+				(hide yes)
+			)
+		)
+	)
 	(global_label "SPI2_IMU_MISO"
 		(shape input)
@@
 			(effects
 				(font
+					(size 1.27 1.27)
+					(italic yes)
+				)
+				(justify right)
+				(hide yes)
+			)
+		)
+	)
+	(global_label "USART1_TX"
+		(shape input)
+		(at 58.42 129.54 180)
+		(fields_autoplaced yes)
+		(effects
+			(font
+				(size 1.27 1.27)
+			)
+			(justify right)
+		)
+		(property "Intersheetrefs" "${INTERSHEET_REFS}"
+			(at 45.2144 129.54 0)
+			(effects
+				(font

Commit message: 18-05-2026
Connections:
- net LED0: no longer U2.38 (PE8)
- net LED1: no longer U2.37 (PE7)
- net USART1_RX: no longer U2.87 (PD6)
- net USART1_TX: no longer U2.86 (PD5)
- new net UART7_RX: U2.37 (PE7)
- new net UART7_TX: U2.38 (PE8)
- new net USART2_RX: U2.87 (PD6)
- new net USART2_TX: U2.86 (PD5)
