File: Vaimanika_H7_Sensor/Vaimanika_H7_Sensor.kicad_sch (KiCad schematic)
At the start: 71 parts, among them SW1 TS-1088-AR02016, U1 TCAN334G, U2 STM32H743VITx, U3 NCP163ASN330T1G, U4 MS5611-01BA, U5 ICM-42688-P, U6 ICM-42688-P, U7 W25Q128JVS, U8 RT9080-33GJ5, U9 BMI088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

Commit message: 20-05-2026
Parts:
- added U10, U11, U12, U13: WAFER-GH1.25-4PWB, New_Library:CONN-SMD_4P-P1.25_XUNPU_WAFER-GH1.25-4PWB, symbol New_Library:WAFER-GH1.25-4PWB
Connections:
- net +5V: now also U10.1, U11.1, U12.1, U13.1
- net GND: now also U10.4, U10.5, U10.6, U11.4, U11.5, U11.6, U12.4, U12.5, U12.6, U13.4, U13.5, U13.6
- net IMU2_CSB2: now also U2.3 (PE4); no longer U2.97 (PE0)
- net UART4_RX: now also U11.3
- net UART4_TX: now also U11.2
- net UART7_RX: now also U12.3
- net UART7_TX: now also U12.2
- net USART2_RX: now also U10.3
- net USART2_TX: now also U10.2
- net UART8_TX: now reaches U2.98 (PE1)
- net UART8_TX: now also U13.2
- new net UART8_RX: U13.3, U2.97 (PE0)

Commit message: 25-05-2026
Parts:
- added TP4, TP5: TestPoint, TestPoint:TestPoint_Pad_D1.0mm, symbol Connector:TestPoint
Connections:
- net GND: now also TP4.1
- net PA15: now reaches U2.77 (PA15)
- net PA15: now also TP5.1

Commit message: 02-06-2026//WFO
Parts:
- U3: LCSC C603656 -> C22435174
Changed lines of the file:
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@@
 			)
 		)
-		(property "LCSC" "C603656"
+		(property "LCSC" "C22435174"
 			(at 165.1 66.04 0)
 			(effects

Commit message: Pilot PCB Done/03-06-2026
Parts:
- C21, C22, C3, C4: LCSC C20539421 -> C53032641
- U3: LCSC C22435174 -> C892187
Connections:
- no-connect marks 10 -> 32
Changed lines of the file:
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@@
 	)
 	(no_connect
+		(at 104.14 175.26)
+	)
+	(no_connect
+		(at 104.14 55.88)
+	)
+	(no_connect
+		(at 58.42 104.14)
+	)
+	(no_connect
+		(at 104.14 83.82)
+	)
+	(no_connect
+		(at 104.14 144.78)
+	)
+	(no_connect
+		(at 104.14 149.86)
+	)
+	(no_connect
 		(at 158.75 215.9)
 	)
 	(no_connect
+		(at 104.14 99.06)
+	)
+	(no_connect
+		(at 58.42 149.86)
+	)
+	(no_connect
+		(at 104.14 71.12)
+	)
+	(no_connect
+		(at 58.42 134.62)
+	)
+	(no_connect
+		(at 104.14 58.42)
+	)
+	(no_connect
 		(at 389.89 67.31)
 	)
 	(no_connect
+		(at 104.14 170.18)
+	)
+	(no_connect
 		(at 158.75 213.36)
 	)
@@
 	)
 	(no_connect
+		(at 58.42 99.06)
+	)
+	(no_connect
 		(at 166.37 41.91)
 	)
 	(no_connect
+		(at 104.14 106.68)
+	)
+	(no_connect
+		(at 58.42 127)
+	)
+	(no_connect
+		(at 104.14 101.6)
+	)
+	(no_connect
+		(at 104.14 86.36)
+	)
+	(no_connect
+		(at 58.42 111.76)
+	)
+	(no_connect
+		(at 104.14 172.72)
+	)
+	(no_connect
 		(at 166.37 34.29)
 	)
@@
 	)
 	(no_connect
+		(at 104.14 104.14)
+	)
+	(no_connect
+		(at 104.14 93.98)
+	)
+	(no_connect
+		(at 58.42 124.46)
+	)
+	(no_connect
 		(at 158.75 166.37)
 	)
@@
 			)
 		)
-		(property "LCSC" "C20539421"
+		(property "LCSC" "C53032641"
 			(at 48.26 160.02 90)
 			(effects
@@
 			)
 		)
-		(property "LCSC" "C20539421"
+		(property "LCSC" "C53032641"
 			(at 48.26 167.64 90)
 			(effects
@@
 			)
 		)
-		(property "LCSC" "C20539421"
+		(property "LCSC" "C53032641"
 			(at 219.71 232.41 0)
 			(effects
@@
 			)
 		)
-		(property "LCSC" "C22435174"
+		(property "LCSC" "C892187"
 			(at 165.1 66.04 0)
 			(effects
@@
 			)
 		)
-		(property "LCSC" "C20539421"
+		(property "LCSC" "C53032641"
 			(at 219.71 185.42 0)
 			(effects
