File: Vaimanika_Rx/Vaimanika_Rx.kicad_sch (KiCad schematic)
At the start: 1 part, among them U1 LR1121IMLTRT

Commit message: 12-05-2026
Parts:
- added C1, C2: 1.2pF, Capacitor_SMD:C_0402_1005Metric, symbol Device:C
- added C3, C4: 1.8pF, Capacitor_SMD:C_0402_1005Metric, symbol Device:C
- added JP1, JP2: U.FL-R-SMT-1, New_Library:RF-SMD_FRF05002-JSS103M, symbol New_Library:U.FL-R-SMT-1
- added L1: 3nH, Inductor_SMD:L_0402_1005Metric, symbol Device:L
- added L2: 4.7nH, Inductor_SMD:L_0402_1005Metric, symbol Device:L
- added U2: RFX2401C, easyeda2kicad:QFN-16_L3.0-W3.0-P0.50-BL-EP1.7, symbol New_Library:RFX2401C
- added U3: SKY13373-460LF, easyeda2kicad:QFN-12_L2.0-W2.0-P0.50-BL-EP, symbol New_Library:SKY13373-460LF
- U1: footprint easyeda2kicad:QFN-32_L5.0-W5.0-P0.50-BL-EP3.7 -> New_Library:QFN-32_L5.0-W5.0-P0.50-BL-EP3.7; LCSC (none) -> C7498014; LCSC Part C7498014 -> (none)
Connections:
- new net: C2.1, JP1.1 (SIG), L1.2
- new net: C4.1, L2.1
- new net: C1.1, L1.1, U3.11 (RFC)
- new net: C3.1, JP2.1 (SIG), L2.2
- new net GND: C1.2, C2.2, C3.2, C4.2, JP1.2 (GND), JP1.3 (GND), JP2.2 (GND), JP2.3 (GND), U3.10 (GND), U3.12 (GND), U3.13 (PAD), U3.7 (GND), U3.8 (GND)
- no-connect marks 0 -> 5
Other:
- note added: "2.4Ghz Link"
- note added: "Sub GHz Link (915 MHz)"
- note added: "Vaimanika Aerospace ELRS Receiver"
- title: (none) -> ELRS Receiver 
- moved on the sheet: U1

Commit message: 14-05-2026
Parts:
- added C5: 10pF, Capacitor_SMD:C_0402_1005Metric, symbol Device:C
- added C6: 4.7uF, Capacitor_SMD:C_0402_1005Metric, symbol Device:C
- added C7: 100nF, Capacitor_SMD:C_0402_1005Metric, symbol Device:C
- added R1, R2: 100K, Resistor_SMD:R_0402_1005Metric, symbol Device:R
- added R3: 220, Resistor_SMD:R_0402_1005Metric, symbol Device:R
- added T1: 0900PC16J0042001E, easyeda2kicad:FILTER-SMD_10P-L2.0-W1.6-BL, symbol New_Library:0900PC16J0042001E
- added U4: ESP32-C3, Package_DFN_QFN:QFN-32-1EP_5x5mm_P0.5mm_EP3.7x3.7mm, symbol MCU_Espressif:ESP32-C3
- added U5: TLV75533PDQNR, easyeda2kicad:X2SON-4_L1.0-W1.0-P0.65-TL-EP, symbol New_Library:TLV75533PDQNR
- added U6: OW2EL89CENUXFMYLC-32M, easyeda2kicad:OSC-SMD_4P-L3.2-W2.5-BL, symbol New_Library:OW2EL89CENUXFMYLC-32M
Connections:
- net GND: now also U1.33 (EP), U2.1 (GND), U2.11 (GND), U2.12 (GND), U2.15 (GND), U2.17 (EP), U2.2 (GND), U2.3 (GND), U2.7 (GND), U2.8 (GND), U2.9 (GND), U3.2 (GND), C6.2, C7.1, R1.2, R2.2, T1.10 (GND), T1.5 (GND), T1.7 (GND), U6.1 (NC), U6.2 (GND)
- net at C4.1, L2.1: now also U3.11 (RFC)
- net at U3.1 (J1): now also T1.6 (RX), T1.8 (TX_LP), T1.9 (TX_HP)
- net at C1.1, L1.1: now also U2.10 (ANT); no longer U3.11 (RFC)
- net GPIO2: now reaches U3.4 (V1)
- net GPIO2: now also U4.6 (GPIO2)
- net GPIO3: now reaches U3.5 (V2)
- net GPIO3: now also U4.8 (GPIO3)
- net at U1.1 (VR_PA): now also C6.1
- net at U1.10 (DIO8): now also R1.1
- net at U1.11 (DIO7): now also R2.1
- net TXEN: now reaches U1.19 (DIO6)
- net TXEN: now also U2.5 (TXEN)
- net +3.3V: now reaches U1.2 (VBAT_RF)
- net +3.3V: now also C7.2
- net RXEN: now reaches U1.20 (DIO5)
- net RXEN: now also U2.6 (RXEN)
- net TXRX: now reaches U1.26 (RFIO_HF)
- net TXRX: now also U2.4 (TXRX)
- net at U1.29 (RFI_N_LF0): now also T1.4 (RFI_N_LFO)
- net at U1.3 (VTCXO): now also U6.4 (VDD)
- net at U1.30 (RFI_P_LF0): now also T1.3 (RFI_P_LFO)
- net at U1.31 (RFO_LP_LF): now also T1.2 (RFO_LP_LF)
- net at U1.32 (RFO_HP_LF): now also T1.1 (RFO_HP_LF)
- net at U1.4 (XTA): now also C5.2
- net RST: now reaches U1.6 (NRESET)
- new net: R3.1, U6.3 (OutPut)
- new net: C5.1, R3.2
- new net: U4.2 (VDD3P3), U4.3 (VDD3P3)
- new net: U4.31 (VDDA), U4.32 (VDDA)
- no-connect marks 5 -> 11
Other:
- moved on the sheet: U1, U2, U3

Commit message: 18-05-2026
Parts:
- removed U4: ESP32-C3, Package_DFN_QFN:QFN-32-1EP_5x5mm_P0.5mm_EP3.7x3.7mm, symbol MCU_Espressif:ESP32-C3
- added C10: 220pF, Capacitor_SMD:C_0402_1005Metric, symbol Device:C
- added C11, C12, C14, C16, C26: 1uF, Capacitor_SMD:C_0402_1005Metric, symbol Device:C
- added C13, C15: 10uF, Capacitor_SMD:C_0402_1005Metric, symbol Device:C
- added C17, C18, C21, C22, C23, C8, C9: 100nF, Capacitor_SMD:C_0402_1005Metric, symbol Device:C
- added C19, C20: 3.3pF, Capacitor_SMD:C_0402_1005Metric, symbol Device:C
- added C24, C25: 12pF, Capacitor_SMD:C_0402_1005Metric, symbol Device:C
- added D1: XL-1010RGBC-WS2812B, New_Library:LED-SMD_4P-L1.0-W1.0-TL_XL-1010RGBC-WS2812B, symbol New_Library:XL-1010RGBC-WS2812B
- added L3: 10uH, Inductor_SMD:L_0603_1608Metric, symbol Device:L
- added L4: 2.2nH, Inductor_SMD:L_0402_1005Metric, symbol Device:L
- added R4, R5, R6, R7: 10K, Resistor_SMD:R_0402_1005Metric, symbol Device:R
- added TP1, TP2: TestPoint, Connector_Wire:SolderWirePad_1x01_SMD_1x2mm, symbol Connector:TestPoint
- added U4: ESP32-C3FH4, New_Library:QFN-32_L5.0-W5.0-P0.50-BL-EP3.7, symbol New_Library:ESP32-C3FH4
- added U7: ANT3216LL00R2400A, New_Library:ANT-SMD_L3.2-W1.6, symbol New_Library:ANT3216LL00R2400A
- added U8: TS2306A 240GF MSM 9_C2976675, New_Library:SW-SMD_4P-L3.0-W2.0-P0.85-LS3.5, symbol New_Library:TS2306A240GFMSM9_C2976675
- added USB1: DEA102700LT-6307A2, New_Library:FILTER-SMD_4P-L1.0-W0.5-L_DEA102700LT-XXX, symbol New_Library:DEA102700LT-6307A2
- added X1: CJ17-400001010B20, easyeda2kicad:CRYSTAL-SMD_4P-L1.6-W1.2-BL, symbol New_Library:CJ17-400001010B20
- T1: footprint easyeda2kicad:FILTER-SMD_10P-L2.0-W1.6-BL -> New_Library:FILTER-SMD_10P-L2.0-W1.6-BL; LCSC (none) -> C19842466; LCSC Part C19842466 -> (none)
- U2: footprint easyeda2kicad:QFN-16_L3.0-W3.0-P0.50-BL-EP1.7 -> New_Library:QFN-16_L3.0-W3.0-P0.50-BL-EP1.7
- U3: footprint easyeda2kicad:QFN-12_L2.0-W2.0-P0.50-BL-EP -> New_Library:QFN-12_L2.0-W2.0-P0.50-BL-EP
- U5: footprint easyeda2kicad:X2SON-4_L1.0-W1.0-P0.65-TL-EP -> New_Library:X2SON-4_L1.0-W1.0-P0.65-TL-EP
Connections:
- net +3.3V: now also U1.15 (VBAT), U2.14 (VDD), U2.16 (VDD), U3.6 (VDD), U5.1 (OUT), C10.1, C11.1, C14.1, C15.1, C16.1, C17.1, C18.1, C21.1, C22.1, C23.1, C9.1, L3.1, R4.1, R5.1, R6.1, R7.1, U4.11 (VDD3P3_RTC), U4.17 (VDD3P3_CPU), U4.18 (VDD_SPI), U4.2 (VDD3P3), U4.3 (VDD3P3), U4.31 (VDDA), U4.32 (VDDA)
- net GND: now also U1.13 (GND), U5.2 (GND), U5.5 (EP), C10.2, C11.2, C12.2, C13.2, C14.2, C15.2, C16.2, C17.2, C18.2, C19.2, C20.2, C21.2, C22.2, C23.2, C24.2, C25.1, C26.1, C8.2, C9.2, D1.3 (GND), U4.33 (EP), U8.2, USB1.2 (GND), USB1.4 (GND), X1.2 (GND), X1.4 (GND)
- net RST: now also R4.2, U4.6 (GPIO2)
- net TXRX: now also USB1.1 (IN); no longer U2.4 (TXRX)
- net +5V: now reaches U5.3 (EN)
- net +5V: now also U5.4 (IN), C12.1, C13.1, D1.2 (VDD)
- net at U1.12 (VREG): now also C8.1
- net at U1.14 (DCC_SW): now also L3.2
- net MISO: now reaches U1.21 (DIO4)
- net MISO: now also U4.12 (MTCK)
- net MOSI: now reaches U1.22 (DIO3)
- net MOSI: now also U4.13 (MTDO)
- net SCK: now reaches U1.23 (DIO2)
- net SCK: now also U4.9 (MTMS)
- net NSS: now reaches U1.24 (DIO1)
- net NSS: now also R7.2, U4.14 (GPIO8)
- net BUSY: now reaches U1.25 (DIO0/BUSY)
- net BUSY: now also U4.8 (GPIO3)
- net DIO1: now reaches U1.9 (DIO9)
- net DIO1: now also U4.10 (MTDI)
- net GPIO2 renamed SKY_V1
- net SKY_V1: now also U4.25 (GPIO18)
- net GPIO3 renamed SKY_V2
- net SKY_V2: now also U4.26 (GPIO19)
- new net: U2.4 (TXRX), USB1.3 (OUT)
- new net: TP2.1, U4.27 (U0RXD)
- new net: C19.1, L4.2, U7.1
- new net: TP1.1, U4.28 (U0TXD)
- new net BUTTON: R6.2, U4.15 (GPIO9), U8.1
- new net CHIP_EN: C26.2, R5.2, U4.7 (CHIP_EN)
- new net DIN: D1.4 (DIN), U4.16 (GPIO10)
- new net LNA_IN: C20.1, L4.1, U4.1 (LNA_IN)
- new net XTAL_N: C24.1, U4.29 (XTAL_N), X1.3
- new net XTAL_P: C25.2, U4.30 (XTAL_P), X1.1
- no-connect marks 11 -> 21
Other:
- moved on the sheet: U5

Commit message: 25-05-2026
Parts:
- U4: LCSC (none) -> C2858491; LCSC Part C2858491 -> (none)
- U5: LCSC (none) -> C2861882; LCSC Part C2861882 -> (none)
- U6: LCSC (none) -> C22434888; LCSC Part C22434888 -> (none)
- U7: LCSC (none) -> C293767; LCSC Part C293767 -> (none)
- U8: LCSC (none) -> C2976675; LCSC Part C2976675 -> (none)
- X1: LCSC (none) -> C2875272; LCSC Part C2875272 -> (none)
Other:
- moved on the sheet: C1, C10, C11, C17, C18, C19, C2, C20, JP1, L1, L4, U2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

Commit message: 25-05-2026
Parts:
- U6: footprint easyeda2kicad:OSC-SMD_4P-L3.2-W2.5-BL -> New_Library:OSC-SMD_4P-L3.2-W2.5-BL
- X1: footprint easyeda2kicad:CRYSTAL-SMD_4P-L1.6-W1.2-BL -> New_Library:CRYSTAL-SMD_4P-L1.6-W1.2-BL
Changed lines of the file:
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@@
 			)
 		)
-		(property "Footprint" "easyeda2kicad:OSC-SMD_4P-L3.2-W2.5-BL"
+		(property "Footprint" "New_Library:OSC-SMD_4P-L3.2-W2.5-BL"
 			(at 100.33 45.72 0)
 			(effects
@@
 				)
 				(justify left)
+				(hide yes)
 			)
 		)
@@
 				)
 				(justify left)
+				(hide yes)
 			)
 		)
@@
 			)
 		)
-		(property "Footprint" "easyeda2kicad:CRYSTAL-SMD_4P-L1.6-W1.2-BL"
+		(property "Footprint" "New_Library:CRYSTAL-SMD_4P-L1.6-W1.2-BL"
 			(at 163.83 36.83 0)
 			(effects

Commit message: 26-05-2026
Parts:
- added C27: 0.3pF, Capacitor_SMD:C_0402_1005Metric, symbol Device:C
Connections:
- net GND: now also C27.1
- net at C1.1, L1.1, U2.10 (ANT): now also C27.2
Changed lines of the file:
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@@
 	)
 	(junction
+		(at 237.49 142.24)
+		(diameter 0)
+		(color 0 0 0 0)
+	)
+	(junction
 		(at 149.86 19.05)
 		(diameter 0)
@@
 	(wire
 		(pts
+			(xy 237.49 124.46) (xy 237.49 125.73)
+		)
+		(stroke
+			(width 0)
+			(type default)
+		)
+	)
+	(wire
+		(pts
 			(xy 231.14 93.98) (xy 233.68 93.98)
 		)
@@
 	(wire
 		(pts
-			(xy 234.95 142.24) (xy 241.3 142.24)
+			(xy 234.95 142.24) (xy 237.49 142.24)
 		)
 		(stroke
@@
 	(wire
 		(pts
+			(xy 237.49 142.24) (xy 241.3 142.24)
+		)
+		(stroke
+			(width 0)
+			(type default)
+		)
+	)
+	(wire
+		(pts
 			(xy 26.67 119.38) (xy 30.48 119.38)
 		)
@@
 	(wire
 		(pts
+			(xy 237.49 133.35) (xy 237.49 142.24)
+		)
+		(stroke
+			(width 0)
+			(type default)
+		)
+	)
+	(wire
+		(pts
 			(xy 204.47 142.24) (xy 204.47 139.7)
 		)
@@
 	)
 	(symbol
+		(lib_id "Device:C")
+		(at 237.49 129.54 0)
+		(unit 1)
+		(exclude_from_sim no)
+		(in_bom yes)
+		(on_board yes)
+		(dnp no)
+		(property "Reference" "C27"
+			(at 233.172 127 0)
+			(effects
+				(font
+					(size 1.27 1.27)
+				)
+				(justify left)
+			)
+		)
+		(property "Value" "0.3pF"
+			(at 238.76 127.254 0)
+			(effects
+				(font
+					(size 1.27 1.27)
+				)
+				(justify left)
+			)
+		)
+		(property "Footprint" "Capacitor_SMD:C_0402_1005Metric"
+			(at 238.4552 133.35 0)
+			(effects
+				(font
+					(size 1.27 1.27)
+				)
+				(hide yes)
+			)
+		)
+		(property "Datasheet" "~"
+			(at 237.49 129.54 0)
+			(effects
+				(font
+					(size 1.27 1.27)
+				)
+				(hide yes)
+			)
+		)
+		(property "Description" "Unpolarized capacitor"
+			(at 237.49 129.54 0)
+			(effects
+				(font
+					(size 1.27 1.27)
+				)
+				(hide yes)
+			)
+		)
+		(property "LCSC" "C1870422"
+			(at 237.49 129.54 0)
+			(effects
+				(font
+					(size 1.27 1.27)
+				)
+				(hide yes)
+			)
+		)
+		(pin "1"
+		)
+		(pin "2"
+		)
+		(instances
+			(project "Vaimanika_Rx"
+				(path "/9053f835-6512-4eb1-a5ab-73d24a49c2c0"
+					(reference "C27")
+					(unit 1)
+				)
+			)
+		)
+	)
+	(symbol
 		(lib_id "power:+3.3V")
 		(at 22.86 77.47 0)
@@
 					(unit 1)
 				)
+			)
+		)
+	)
+	(symbol
+		(lib_id "power:GND")
+		(at 237.49 124.46 180)
+		(unit 1)
+		(exclude_from_sim no)
+		(in_bom yes)
+		(on_board yes)
+		(dnp no)
+		(fields_autoplaced yes)
+		(property "Reference" "#PWR063"
+			(at 237.49 118.11 0)
+			(effects
+				(font
+					(size 1.27 1.27)
+				)
+				(hide yes)
+			)
+		)
+		(property "Value" "GND"
+			(at 237.49 119.38 0)
+			(effects
+				(font
+					(size 1.27 1.27)
+				)
+				(hide yes)
+			)
+		)
+		(property "Footprint" ""
+			(at 237.49 124.46 0)
+			(effects
+				(font
+					(size 1.27 1.27)
+				)
+				(hide yes)
+			)
+		)
+		(property "Datasheet" ""
+			(at 237.49 124.46 0)
+			(effects
+				(font
+					(size 1.27 1.27)
+				)
+				(hide yes)
+			)
+		)
+		(property "Description" "Power symbol creates a global label with name \"GND\" , ground"
+			(at 237.49 124.46 0)
+			(effects
+				(font
+					(size 1.27 1.27)
+				)
+				(hide yes)
+			)
+		)
+		(pin "1"
+		)
+		(instances
+			(project "Vaimanika_Rx"
+				(path "/9053f835-6512-4eb1-a5ab-73d24a49c2c0"
+					(reference "#PWR063")
+					(unit 1)
+				)

Commit message: 26-05-2026
Connections:
- net at T1.9 (TX_HP), U3.1 (J1): no longer T1.6 (RX), T1.8 (TX_LP)
- net at U3.3 (J3): now also T1.6 (RX)
Changed lines of the file:
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@@
-	)
-	(junction
-		(at 184.15 96.52)
-		(diameter 0)
-		(color 0 0 0 0)
 	)
 	(junction
@@
 	(junction
 		(at 63.5 107.95)
-		(diameter 0)
-		(color 0 0 0 0)
-	)
-	(junction
-		(at 184.15 101.6)
 		(diameter 0)
 		(color 0 0 0 0)
@@
 	)
 	(no_connect
+		(at 184.15 96.52)
+	)
+	(no_connect
 		(at 67.31 45.72)
 	)
@@
 	)
 	(no_connect
-		(at 215.9 83.82)
-	)
-	(no_connect
 		(at 100.33 77.47)
 	)
@@
 	(wire
 		(pts
-			(xy 220.98 83.82) (xy 220.98 81.28)
-		)
-		(stroke
-			(width 0)
-			(type default)
-		)
-	)
-	(wire
-		(pts
 			(xy 15.24 49.53) (xy 15.24 50.8)
 		)
@@
 	(wire
 		(pts
-			(xy 182.88 93.98) (xy 184.15 93.98)
+			(xy 182.88 93.98) (xy 194.31 93.98)
 		)
 		(stroke
@@
 	(wire
 		(pts
-			(xy 191.77 101.6) (xy 184.15 101.6)
-		)
-		(stroke
-			(width 0)
-			(type default)
-		)
-	)
-	(wire
-		(pts
 			(xy 199.39 134.62) (xy 199.39 135.89)
 		)
@@
 	(wire
 		(pts
+			(xy 215.9 80.01) (xy 215.9 83.82)
+		)
+		(stroke
+			(width 0)
+			(type default)
+		)
+	)
+	(wire
+		(pts
 			(xy 269.24 31.75) (xy 262.89 31.75)
 		)
@@
 	(wire
 		(pts
-			(xy 182.88 101.6) (xy 184.15 101.6)
+			(xy 182.88 101.6) (xy 191.77 101.6)
 		)
 		(stroke
@@
 	(wire
 		(pts
+			(xy 194.31 82.55) (xy 220.98 82.55)
+		)
+		(stroke
+			(width 0)
+			(type default)
+		)
+	)
+	(wire
+		(pts
 			(xy 67.31 25.4) (xy 67.31 27.94)
 		)
@@
 	(wire
 		(pts
-			(xy 184.15 93.98) (xy 184.15 96.52)
-		)
-		(stroke
-			(width 0)
-			(type default)
-		)
-	)
-	(wire
-		(pts
 			(xy 257.81 99.06) (xy 257.81 96.52)
 		)
@@
 	(wire
 		(pts
+			(xy 194.31 93.98) (xy 194.31 82.55)
+		)
+		(stroke
+			(width 0)
+			(type default)
+		)
+	)
+	(wire
+		(pts
 			(xy 110.49 34.29) (xy 110.49 31.75)
 		)
@@
 	(wire
 		(pts
-			(xy 191.77 81.28) (xy 191.77 101.6)
+			(xy 191.77 80.01) (xy 191.77 101.6)
 		)
 		(stroke
@@
 	(wire
 		(pts
-			(xy 184.15 101.6) (xy 184.15 96.52)
-		)
-		(stroke
-			(width 0)
-			(type default)
-		)
-	)
-	(wire
-		(pts
 			(xy 204.47 137.16) (xy 204.47 139.7)
 		)
@@
 	(wire
 		(pts
+			(xy 220.98 83.82) (xy 220.98 82.55)
+		)
+		(stroke
+			(width 0)
+			(type default)
+		)
+	)
+	(wire
+		(pts
 			(xy 69.85 97.79) (xy 69.85 109.22)
 		)
@@
 	(wire
 		(pts
-			(xy 220.98 81.28) (xy 191.77 81.28)
-		)
-		(stroke
-			(width 0)
-			(type default)
-		)
-	)
-	(wire
-		(pts
 			(xy 107.95 76.2) (xy 107.95 77.47)
 		)
@@
 		)
 		(stroke
+			(width 0)
+			(type default)
+		)
+	)
+	(wire
+		(pts
+			(xy 191.77 80.01) (xy 215.9 80.01)
+		)
+		(stroke

Commit message: 28-05-2026
Parts:
- removed C14: 1uF, Capacitor_SMD:C_0402_1005Metric, symbol Device:C
- removed C15: 10uF, Capacitor_SMD:C_0402_1005Metric, symbol Device:C
- removed TP1, TP2: TestPoint, Connector_Wire:SolderWirePad_1x01_SMD_1x2mm, symbol Connector:TestPoint
- removed U5: TLV75533PDQNR, New_Library:X2SON-4_L1.0-W1.0-P0.65-TL-EP, symbol New_Library:TLV75533PDQNR
- added J1: Conn_01x04, New_Library:Rec_Conn_01x04, symbol Connector_Generic:Conn_01x04
- added U9: CJ6109B33M, New_Library:SOT-23-5_L2.9-W1.6-P0.95-LS2.8-BR, symbol New_Library:CJ6109B33M
- C12: value 1uF -> 4.7uF; LCSC C5137474 -> C22399610
- C13: value 10uF -> 4.7uF; LCSC C7472949 -> C22399610
Connections:
- net +3.3V: now also C13.1, U9.5 (VOUT)
- net +5V: now also J1.1 (Pin_1), U9.1 (VIN), U9.3 (CE); no longer C13.1
- net GND: now also J1.4 (Pin_4), U9.2 (VSS)
- net U0RXD: now reaches U4.27 (U0RXD)
- net U0RXD: now also J1.2 (Pin_2)
- net U0TXD: now reaches U4.28 (U0TXD)
- net U0TXD: now also J1.3 (Pin_3)
- no-connect marks 21 -> 22
Other:
- moved on the sheet: C12, C13
