File: Vaimanika_Rx/Vaimanika_Rx.kicad_sch (KiCad schematic)
At the start: 51 parts, among them J1 Conn_01x04, T1 0900PC16J0042001E, U1 LR1121IMLTRT, U2 RFX2401C, U3 SKY13373-460LF, U4 ESP32-C3FH4, U6 OW2EL89CENUXFMYLC-32M, U7 ANT3216LL00R2400A, U8 TS2306A 240GF MSM 9_C2976675, U9 CJ6109B33M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

Commit message: 02-06-2026//WFO
Parts:
- C10: LCSC C20069331 -> C597026
- C17, C18, C21, C22, C23: LCSC C5137468 -> C237172
- C3, C4: LCSC C5186870 -> C301970
- C7, C8, C9: LCSC C7393848 -> C237172
- R4, R5, R6, R7: LCSC C60489 -> C22404129
Changed lines of the file:
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@@
 				)
 				(justify left)
-				(hide yes)
 			)
 		)
@@
 				)
 				(justify left)
-				(hide yes)
 			)
 		)
@@
 			)
 		)
-		(property "LCSC" "C5137468"
+		(property "LCSC" "C237172"
 			(at 48.26 88.9 0)
 			(effects
@@
 			)
 		)
-		(property "LCSC" "C5137468"
+		(property "LCSC" "C237172"
 			(at 81.28 64.77 0)
 			(effects
@@
 			)
 		)
-		(property "LCSC" "C5186870"
+		(property "LCSC" "C301970"
 			(at 240.03 102.87 0)
 			(effects
@@
 			)
 		)
-		(property "LCSC" "C5137468"
+		(property "LCSC" "C237172"
 			(at 73.66 64.77 0)
 			(effects
@@
 			)
 		)
-		(property "LCSC" "C60489"
+		(property "LCSC" "C22404129"
 			(at 19.05 85.09 0)
 			(effects
@@
 			)
 		)
-		(property "LCSC" "C60489"
+		(property "LCSC" "C22404129"
 			(at 26.67 114.3 0)
 			(effects
@@
 			)
 		)
-		(property "LCSC" "C60489"
+		(property "LCSC" "C22404129"
 			(at 26.67 130.81 0)
 			(effects
@@
 			)
 		)
-		(property "LCSC" "C5186870"
+		(property "LCSC" "C301970"
 			(at 257.81 102.87 0)
 			(effects
@@
 			)
 		)
-		(property "LCSC" "C7393848"
+		(property "LCSC" "C237172"
 			(at 120.65 62.23 90)
 			(effects
@@
 			)
 		)
-		(property "LCSC" "C7393848"
+		(property "LCSC" "C237172"
 			(at 69.85 113.03 90)
 			(effects
@@
 			)
 		)
-		(property "LCSC" "C5137468"
+		(property "LCSC" "C237172"
 			(at 54.61 88.9 0)
 			(effects
@@
 			)
 		)
-		(property "LCSC" "C7393848"
+		(property "LCSC" "C237172"
 			(at 73.66 120.65 90)
 			(effects
@@
 			)
 		)
-		(property "LCSC" "C5137468"
+		(property "LCSC" "C237172"
 			(at 15.24 54.61 0)
 			(effects
@@
 			)
 		)
-		(property "LCSC" "C20069331"
+		(property "LCSC" "C597026"
 			(at 204.47 130.81 0)
 			(effects
@@
 			)
 		)
-		(property "LCSC" "C60489"
+		(property "LCSC" "C22404129"
 			(at 26.67 85.09 0)
 			(effects

Commit message: Pilot PCB Done/03-06-2026
Parts:
- C17, C18, C21, C22, C23, C7, C8, C9: LCSC C237172 -> C60474
- J1: now left out of the parts list
Changed lines of the file:
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@@
 			)
 		)
-		(property "LCSC" "C237172"
+		(property "LCSC" "C60474"
 			(at 48.26 88.9 0)
 			(effects
@@
 			)
 		)
-		(property "LCSC" "C237172"
+		(property "LCSC" "C60474"
 			(at 81.28 64.77 0)
 			(effects
@@
 			)
 		)
-		(property "LCSC" "C237172"
+		(property "LCSC" "C60474"
 			(at 73.66 64.77 0)
 			(effects
@@
 		(unit 1)
 		(exclude_from_sim no)
-		(in_bom yes)
+		(in_bom no)
 		(on_board yes)
 		(dnp no)
@@
 			)
 		)
-		(property "LCSC" "C237172"
+		(property "LCSC" "C60474"
 			(at 120.65 62.23 90)
 			(effects
@@
 			)
 		)
-		(property "LCSC" "C237172"
+		(property "LCSC" "C60474"
 			(at 69.85 113.03 90)
 			(effects
@@
 			)
 		)
-		(property "LCSC" "C237172"
+		(property "LCSC" "C60474"
 			(at 54.61 88.9 0)
 			(effects
@@
 			)
 		)
-		(property "LCSC" "C237172"
+		(property "LCSC" "C60474"
 			(at 73.66 120.65 90)
 			(effects
@@
 			)
 		)
-		(property "LCSC" "C237172"
+		(property "LCSC" "C60474"
 			(at 15.24 54.61 0)
 			(effects
