File: Vaimanika_Rx/Vaimanika_Rx.kicad_pcb (KiCad board)
At the start: 4 copper layers, 18 x 25 mm, 53 parts, among them T1 0900PC16J0042001E, U1 LR1121IMLTRT, U2 RFX2401C, U3 SKY13373-460LF, U4 ESP32-C3FH4, U5 TLV75533PDQNR, U6 OW2EL89CENUXFMYLC-32M, U7 ANT3216LL00R2400A, U8 TS2306A 240GF MSM 9_C2976675, X1 CJ17-400001010B20

Commit message: 26-05-2026
Parts:
- added C27: 0.3pF, Capacitor_SMD:C_0402_1005Metric, F.Cu at (152.1, 94.8)
- moved U3 71.3 mm to (145.9, 97.2)
Routing:
- net Net-(U3-RFC): track 1.08 -> 7.03 mm
- net GND: track 11.6 -> 16.6 mm
- net Net-(U2-ANT): track 5.82 -> 7.48 mm
- added copper zone on In2.Cu, net GND

Commit message: 26-05-2026
Parts:
- C10, C11: moved to B.Cu
- moved U1 91.0 mm to (146.8, 105.2), turned to -90 degrees
- moved C10 88.2 mm to (150.3, 98.0)
- moved C11 87.6 mm to (150.3, 96.9)
- moved USB1 85.9 mm to (150.3, 100.7)
- moved T1 73.6 mm to (145.8, 100.6)
- moved U2 0.85 mm to (151.3, 97.2)
- moved C27 0.85 mm to (153.0, 94.8)
Connections:
- T1 pad 8: Net-(T1-RX) -> unconnected-(T1-TX_LP-Pad8)
- T1 pad 9: Net-(T1-RX) -> Net-(T1-TX_HP)
- U3 pad 1: Net-(T1-RX) -> Net-(T1-TX_HP)
- U3 pad 3: unconnected-(U3-J3-Pad3) -> Net-(T1-RX)
Routing:
- net GND: track 16.6 -> 6.41 mm
- net Net-(U3-RFC): track 7.03 -> 3.38 mm
- net VDD3P3: track 0.00 -> 3.23 mm, vias 0 -> 3
- net TXRX: track 0.00 -> 2.98 mm
- net Net-(U2-TXRX): track 0.00 -> 2.71 mm
- net Net-(T1-TX_HP): track 0.00 -> 1.86 mm
- net Net-(T1-RX): track 0.00 -> 1.81 mm
- net Net-(T1-RFO_LP_LF): track 0.00 -> 1.33 mm
- net Net-(T1-RFO_HP_LF): track 0.00 -> 1.33 mm
- net Net-(T1-RFI_P_LFO): track 0.00 -> 1.33 mm
- net Net-(T1-RFI_N_LFO): track 0.00 -> 1.33 mm

Commit message: 27-05-2026
Parts:
- C10, C11: moved to F.Cu
- moved D1 64.0 mm to (124.7, 99.4)
- moved L3 53.6 mm to (119.6, 100.9)
- moved U4 52.9 mm to (114.1, 98.3)
- moved C22 51.8 mm to (117.8, 93.8)
- moved TP1 51.2 mm to (123.2, 84.8)
- moved TP2 51.2 mm to (125.6, 84.8)
- moved C23 51.1 mm to (120.6, 84.0)
- moved C24 51.1 mm to (120.6, 86.0)
- moved C25 51.1 mm to (120.6, 87.9)
- moved C26 51.1 mm to (120.6, 89.9)
- moved C15 51.1 mm to (114.9, 91.9)
- moved C16 51.1 mm to (114.9, 93.8)
- moved C17 50.8 mm to (117.8, 84.0)
- moved C18 50.8 mm to (117.8, 86.0)
- moved C19 50.8 mm to (117.8, 87.9)
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Routing:
- net Net-(U3-RFC): track 3.38 -> 7.03 mm
- net TXRX: track 2.98 -> 0.00 mm
- net GND: vias 0 -> 1
- removed copper zone on In2.Cu, net GND
Other:
- board text removed: "ELRS Reciver"
- board text removed: "Vaimanika Aerospace ELRS Receiver"

Commit message: 27-05-2026
Parts:
- C16, C19, C20, C24, C25, C26, L4, R4, R5, U4, U7, X1: moved to B.Cu
- moved L4 38.3 mm to (144.7, 98.4), turned to 180 degrees
- moved U4 36.5 mm to (150.5, 95.1), turned to 90 degrees
- moved R6 35.7 mm to (144.7, 99.1), turned to 180 degrees
- moved R4 35.7 mm to (144.7, 94.4)
- moved R5 35.6 mm to (144.8, 93.4)
- moved C21 34.5 mm to (152.0, 95.6), turned to 180 degrees
- moved C24 34.4 mm to (150.5, 103.1), turned to -90 degrees
- moved C22 34.3 mm to (152.0, 94.5), turned to 180 degrees
- moved C23 32.1 mm to (152.1, 90.3)
- moved C16 32.0 mm to (146.6, 98.2), turned to 90 degrees
- moved C25 30.9 mm to (147.6, 103.1), turned to 90 degrees
- moved C19 29.2 mm to (144.6, 99.5)
- moved C20 27.9 mm to (144.6, 97.3), turned to 180 degrees
- moved X1 24.6 mm to (149.1, 101.0), turned to 45 degrees
- moved U7 24.5 mm to (144.7, 102.5), turned to -90 degrees
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Routing:
- net VDD3P3: track 3.23 -> 33.4 mm, vias 3 -> 7
- net SCK: track 0.00 -> 28.7 mm, vias 0 -> 1
- net MISO: track 0.00 -> 27.1 mm, vias 0 -> 1
- net MOSI: track 0.00 -> 23.8 mm, vias 0 -> 1
- net BUTTON: track 0.00 -> 23.6 mm, vias 0 -> 2
- net NSS: track 0.00 -> 18.7 mm, vias 0 -> 1
- net SKY_V2: track 0.00 -> 6.08 mm, vias 0 -> 1
- net RXEN: track 0.00 -> 5.99 mm, vias 0 -> 2
- net XTAL_N: track 0.00 -> 5.87 mm
- net XTAL_P: track 0.00 -> 5.79 mm
- net TXEN: track 0.00 -> 5.00 mm, vias 0 -> 2
- net DIN: track 0.00 -> 4.14 mm, vias 0 -> 1
- net CHIP_EN: track 0.00 -> 4.03 mm
- net LNA_IN: track 0.00 -> 4.02 mm
- net TXRX: track 0.00 -> 3.06 mm
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
Commit message: 28-05-2026
Parts:
- removed C14: 1uF, Capacitor_SMD:C_0402_1005Metric
- removed C15: 10uF, Capacitor_SMD:C_0402_1005Metric
- removed TP1, TP2: TestPoint, Connector_Wire:SolderWirePad_1x01_SMD_1x2mm
- removed U5: TLV75533PDQNR, New_Library:X2SON-4_L1.0-W1.0-P0.65-TL-EP
- added J1: Conn_01x04, New_Library:Rec_Conn_01x04, F.Cu at (152.0, 113.2)
- added U9: CJ6109B33M, New_Library:SOT-23-5_L2.9-W1.6-P0.95-LS2.8-BR, B.Cu at (153.4, 107.7)
- C11, R6, R7: moved to B.Cu
- C12: value 1uF -> 4.7uF; moved to B.Cu
- C13: value 10uF -> 4.7uF; moved to B.Cu
- moved C9 48.5 mm to (156.8, 110.4), turned to -90 degrees
- moved R2 47.9 mm to (151.5, 110.4), turned to -90 degrees
- moved R1 47.9 mm to (150.4, 110.4), turned to -90 degrees
- moved R7 46.5 mm to (155.5, 101.0), turned to -90 degrees
- moved C8 45.4 mm to (152.6, 110.4), turned to -90 degrees
- moved C12 43.4 mm to (153.9, 105.0), turned to 90 degrees
- moved C10 43.2 mm to (154.8, 100.0), turned to -135 degrees
- moved C5 43.0 mm to (148.7, 106.5), turned to 90 degrees
- moved C11 43.0 mm to (154.4, 100.9), turned to -90 degrees
- moved R3 41.9 mm to (147.6, 106.6), turned to -90 degrees
- moved C13 41.4 mm to (152.6, 105.0), turned to 90 degrees
- moved C6 37.9 mm to (146.5, 101.6), turned to 180 degrees
- moved C7 37.5 mm to (146.5, 102.7)
- moved L3 36.4 mm to (154.7, 110.6), turned to 180 degrees
- moved D1 35.1 mm to (159.1, 110.3)
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Connections:
- C13 pad 1: +5V -> VDD3P3
- U4 pad 27: Net-(U4-U0RXD) -> U0RXD
- U4 pad 28: Net-(U4-U0TXD) -> U0TXD
Routing:
- net VDD3P3: track 33.4 -> 65.0 mm, vias 7 -> 13
- net DIO1: track 2.30 -> 24.5 mm, vias 1 -> 2
- net RST: track 2.69 -> 20.8 mm, vias 0 -> 2
- net +5V: track 0.00 -> 16.6 mm, vias 0 -> 1
- net BUSY: track 0.00 -> 15.8 mm, vias 0 -> 2
- net BUTTON: track 23.6 -> 11.8 mm
- net GND: track 8.66 -> 15.8 mm, vias 8 -> 11
- net Net-(U1-VTCXO): track 0.00 -> 4.65 mm
- net Net-(U1-VR_PA): track 0.00 -> 4.43 mm
- net RXEN: track 5.99 -> 3.34 mm
- net Net-(U1-DIO8): track 0.00 -> 2.36 mm
- net TXEN: track 5.00 -> 2.67 mm
- net Net-(U1-DCC_SW): track 0.00 -> 2.31 mm
- net Net-(U1-XTA): track 0.00 -> 1.96 mm
- net Net-(U1-DIO7): track 0.00 -> 1.86 mm
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
Commit message: 30-05-2026//WFO
Parts:
- moved R6 2.65 mm to (144.8, 112.0)
- moved C12 0.65 mm to (154.5, 105.0)
- moved C21 0.54 mm to (152.6, 95.6)
- moved C22 0.54 mm to (152.6, 94.5)
- moved L3 0.36 mm to (154.7, 110.2)
- moved U8 0.33 mm to (144.9, 110.9)
Routing:
- net U0RXD: track 1.19 -> 21.3 mm
- net U0TXD: track 1.17 -> 21.1 mm
- net VDD3P3: track 65.0 -> 60.4 mm, vias 13 -> 10
- net BUTTON: track 11.8 -> 10.2 mm
- net GND: vias 11 -> 20
Other:
- board text added: "+5V"
- board text added: "G"

Commit message: 02-06-2026//WFO
Parts:
- added G***: LOGO, LOGO, B.Cu at (158.2, 111.3)
Routing:
- net BUTTON: track 10.2 -> 41.4 mm
- net VDD3P3: track 60.4 -> 89.0 mm, vias 10 -> 12
- net DIN: track 5.10 -> 21.3 mm
- net RXEN: track 3.34 -> 14.7 mm
- net TXEN: track 2.67 -> 13.8 mm, vias 2 -> 0
- net GND: track 15.8 -> 18.9 mm, vias 20 -> 30
Other:
- board size 18 x 25 mm -> 18 x 25.5 mm
- board text added: "Rx"
- board text added: "Tx"

Commit message: Pilot PCB Done/03-06-2026
Parts:
- added G***: LOGO, LOGO, F.Cu at (148.4, 96.8)
- added G***: LOGO, LOGO, B.Cu at (146.3, 105.9)
- moved G*** 0.47 mm to (158.0, 110.9)
Routing:
- net GND: vias 30 -> 32
Other:
- board text added: "VEG LINK"
